File: hardware/orion_cpu/orion_cpu.kicad_pcb (KiCad board)
At the start: 2 copper layers, 99.7 x 99.7 mm, 49 parts, among them J1 C96ABC, SW1 CONFIG, SW2 ROM1

Commit message: Обновлён проект платы процессорного модуля
Parts:
- added C21: 100n, Capacitor_SMD:C_0805_2012Metric, B.Cu at (77.5, 52.1)
- added C22: 100n, Capacitor_SMD:C_0805_2012Metric, B.Cu at (159.8, 99.9)
- added J2: JTAG, Connector_PinHeader_2.54mm:PinHeader_2x05_P2.54mm_Vertical, F.Cu at (77.5, 55.2)
- added R13: 1K, Resistor_SMD:R_0805_2012Metric, B.Cu at (162.6, 73.7)
- added R14: 1K, Resistor_SMD:R_0805_2012Metric, B.Cu at (162.6, 99.1)
- added R15: 1K, Resistor_SMD:R_0805_2012Metric, B.Cu at (162.6, 91.4)
- added R16: 1K, Resistor_SMD:R_0805_2012Metric, B.Cu at (162.6, 88.9)
- added R17: 1K, Resistor_SMD:R_0805_2012Metric, B.Cu at (162.6, 86.4)
- added R18: 1K, Resistor_SMD:R_0805_2012Metric, B.Cu at (162.6, 83.8)
- added R19: 1K, Resistor_SMD:R_0805_2012Metric, B.Cu at (162.6, 81.3)
- added R20: 1K, Resistor_SMD:R_0805_2012Metric, B.Cu at (162.6, 78.7)
- added R21: 1K, Resistor_SMD:R_0805_2012Metric, B.Cu at (162.6, 76.2)
- added R22: 1K, Resistor_SMD:R_0805_2012Metric, F.Cu at (111.1, 54.6)
- added R23: 1K, Resistor_SMD:R_0805_2012Metric, F.Cu at (143.5, 99.1)
- added R24: 1K, Resistor_SMD:R_0805_2012Metric, F.Cu at (145.4, 96.5)
- added R25: 1K, Resistor_SMD:R_0805_2012Metric, F.Cu at (139.7, 101.0)
- added R26: 1K, Resistor_SMD:R_0805_2012Metric, F.Cu at (141.6, 97.2)
- added R27: 1K, Resistor_SMD:R_0805_2012Metric, F.Cu at (148.6, 97.8)
- added R28: 1K, Resistor_SMD:R_0805_2012Metric, B.Cu at (116.2, 123.2)
- added R29: 1K, Resistor_SMD:R_0805_2012Metric, B.Cu at (74.3, 62.9)
- added R30: 1K, Resistor_SMD:R_0805_2012Metric, B.Cu at (74.3, 60.3)
- added R31: 1K, Resistor_SMD:R_0805_2012Metric, B.Cu at (74.3, 65.4)
- added R32: 1K, Resistor_SMD:R_0805_2012Metric, B.Cu at (74.3, 55.2)
- added R33: 1K, Resistor_SMD:R_0805_2012Metric, B.Cu at (140.3, 123.2)
- added SW3: RESET, Buttons_Switches_ThroughHole:SW_PUSH_6mm, F.Cu at (160.7, 127.0)
- C1, C10, C12, C2, C3, C4, C5, C6, C7, C8, C9, DD10: moved to B.Cu
- DD11: value AP6 -> 74AHCT1G04; footprint Package_SO:SOIC-20W_7.5x12.8mm_P1.27mm -> Package_TO_SOT_SMD:SOT-353_SC-70-5_Handsoldering; moved to F.Cu
- DD6, DD7, DD8, DD9: value AS7C4098A -> CY7C1049B; footprint Projects:SOJ-44 -> Projects:SOJ-36
- moved C9 88.7 mm to (119.1, 71.9), turned to 90 degrees
- moved C5 84.1 mm to (121.2, 78.5), turned to 270 degrees
- moved C4 83.3 mm to (118.6, 78.5), turned to 270 degrees
- moved C2 83.0 mm to (115.6, 71.9), turned to 90 degrees
- moved C3 82.9 mm to (115.6, 78.5), turned to 90 degrees
- moved C8 82.3 mm to (122.2, 71.9), turned to 90 degrees
- moved C7 75.9 mm to (125.2, 71.9), turned to 270 degrees
- moved C6 73.9 mm to (123.4, 78.5), turned to 270 degrees
- moved C1 51.3 mm to (154.9, 86.4), turned to 270 degrees
- moved DD11 26.4 mm to (115.6, 55.2), turned to 180 degrees
- moved C10 25.8 mm to (74.4, 127.3), turned to 180 degrees
- moved C11 24.2 mm to (106.7, 121.7), turned to 270 degrees
- moved C12 22.9 mm to (132.6, 121.7), turned to 270 degrees
- moved DD6 4.45 mm to (85.7, 105.4)
- moved DD7 4.45 mm to (85.7, 95.2)
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Connections:
- net /R3 renamed /R0
- net Net-(DD2-Pad71) renamed /r2
- net Net-(DD2-Pad88) renamed /R1
- DD10 pad 3: /MD6 -> /MD0
- DD10 pad 4: /MD5 -> /MD6
- DD10 pad 5: /MD4 -> /MD1
- DD10 pad 6: /MD3 -> /MD2
- DD10 pad 7: /MD2 -> /MD5
- DD10 pad 8: /MD1 -> /MD3
- DD10 pad 9: /MD0 -> /MD4
- DD11 pad 1: /~MWR -> (no net)
- DD11 pad 2: /MD15 -> /MA16
- DD11 pad 3: /MD14 -> GND
- DD11 pad 4: /MD13 -> /~UB
- DD11 pad 5: /MD12 -> VCC
- DD12 pad 10: /~IRQS -> /~IRQ7
- DD12 pad 11: Net-(DD12-Pad11) -> /~IRQS
- DD12 pad 2: /~M1 -> /~INT
- DD12 pad 23: /~INT -> Net-(DD12-Pad23)
- DD12 pad 3: /~IRQ1 -> /~M1
- DD12 pad 4: /~IRQ2 -> /~IRQ1
- DD12 pad 5: /~IRQ3 -> /~IRQ2
- DD12 pad 6: /~IRQ4 -> /~IRQ3
- DD12 pad 7: /~IRQ5 -> /~IRQ4
- DD12 pad 8: /~IRQ6 -> /~IRQ5
- DD12 pad 9: /~IRQ7 -> /~IRQ6
- DD2 pad 1: /MA16 -> /MA17
- DD2 pad 100: /MA15 -> /~VO0
- DD2 pad 2: /MA17 -> /MA18
- DD2 pad 46: /D2 -> /D6
- DD2 pad 47: /A0 -> /D5
- DD2 pad 48: /A1 -> /D4
- DD2 pad 49: /D6 -> /D3
- DD2 pad 50: /A2 -> /D2
- DD2 pad 52: Net-(DD2-Pad52) -> /A0
- DD2 pad 53: Net-(DD2-Pad53) -> /A1
- DD2 pad 54: Net-(DD2-Pad54) -> /A2
- DD2 pad 55: Net-(DD2-Pad55) -> /A3
- DD2 pad 56: Net-(DD2-Pad56) -> /A4
- DD2 pad 57: Net-(DD2-Pad57) -> /A5
- DD2 pad 58: Net-(DD2-Pad58) -> /A6
- DD2 pad 60: Net-(DD2-Pad60) -> /ZA15
- DD2 pad 61: Net-(DD2-Pad61) -> /A7
- DD2 pad 63: Net-(DD2-Pad63) -> /ZA14
- DD2 pad 64: Net-(DD2-Pad64) -> /A8
- DD2 pad 65: Net-(DD2-Pad65) -> /A13
- DD2 pad 67: Net-(DD2-Pad67) -> /A9
- DD2 pad 68: Net-(DD2-Pad68) -> /A12
- DD2 pad 69: Net-(DD2-Pad69) -> /A10
- DD2 pad 70: Net-(DD2-Pad70) -> /A11
- DD2 pad 72: Net-(DD2-Pad72) -> /~TRB
- DD2 pad 75: Net-(DD2-Pad75) -> /INT50
- DD2 pad 76: Net-(DD2-Pad76) -> /SND
- DD2 pad 78: Net-(DD2-Pad78) -> /~OE0
- DD2 pad 79: Net-(DD2-Pad79) -> /MA14
- DD2 pad 80: Net-(DD2-Pad80) -> /A14
- DD2 pad 81: Net-(DD2-Pad81) -> /MA15
- DD2 pad 83: Net-(DD2-Pad83) -> /A15
- DD2 pad 85: Net-(DD2-Pad85) -> /MA16
- DD2 pad 89: /R2 -> /~BLIO
- DD2 pad 92: Net-(DD2-Pad92) -> /~VCE
- DD2 pad 93: Net-(DD2-Pad93) -> /~MWR
- DD2 pad 94: /~MWR -> /~MRD
- DD2 pad 96: /~LB -> /pFA
- DD2 pad 97: /~UB -> /pF8
- DD2 pad 98: /~MRD -> /pFC
- DD2 pad 99: /MA14 -> /~VO1
- DD4 pad 31: /PGM1 -> Net-(DD4-Pad31)
- DD5 pad 31: /PGM2 -> Net-(DD5-Pad31)
- DD6 pad 1: /MA17 -> /MA18
- DD6 pad 10: /MD3 -> GND
- DD6 pad 11: VCC -> /MD2
- DD6 pad 12: GND -> /MD3
- DD6 pad 13: /MD4 -> /~MWR
- DD6 pad 14: /MD5 -> /A0
- DD6 pad 15: /MD6 -> /A2
- DD6 pad 16: /MD7 -> /A4
- DD6 pad 17: /~MWR -> /A6
- DD6 pad 18: /A0 -> /A12
- DD6 pad 19: /A2 -> (no net)
- DD6 pad 2: /MA16 -> /MA17
- DD6 pad 20: /A4 -> /A7
- DD6 pad 21: /A6 -> /A5
- DD6 pad 22: /A12 -> /A3
- DD6 pad 23: /A7 -> /A1
- DD6 pad 24: /A5 -> /A8
- DD6 pad 25: /A3 -> /MD4
- DD6 pad 26: /A1 -> /MD5
- DD6 pad 27: /A8 -> VCC
- DD6 pad 28: (no net) -> GND
- DD6 pad 29: /MD8 -> /MD6
- DD6 pad 30: /MD9 -> /MD7
- DD6 pad 31: /MD10 -> /~MRD
- DD6 pad 32: /MD11 -> /A11
- DD6 pad 33: VCC -> /A9
- DD6 pad 34: GND -> /A10
- DD6 pad 35: /MD12 -> /MA16
- DD6 pad 36: /MD13 -> (no net)
- DD6 pad 9: /MD2 -> VCC
- DD7 pad 1: /MA17 -> /MA18
- DD7 pad 10: /MD3 -> GND
- DD7 pad 11: VCC -> /MD2
- DD7 pad 12: GND -> /MD3
- DD7 pad 13: /MD4 -> /~MWR
- DD7 pad 14: /MD5 -> /A0
- DD7 pad 15: /MD6 -> /A2
- DD7 pad 16: /MD7 -> /A4
- DD7 pad 17: /~MWR -> /A6
- DD7 pad 18: /A0 -> /A12
- DD7 pad 19: /A2 -> (no net)
- DD7 pad 2: /MA16 -> /MA17
- DD7 pad 20: /A4 -> /A7
- DD7 pad 21: /A6 -> /A5
- DD7 pad 22: /A12 -> /A3
- DD7 pad 23: /A7 -> /A1
- DD7 pad 24: /A5 -> /A8
- DD7 pad 25: /A3 -> /MD4
- DD7 pad 26: /A1 -> /MD5
- DD7 pad 27: /A8 -> VCC
- DD7 pad 28: (no net) -> GND
- DD7 pad 29: /MD8 -> /MD6
- DD7 pad 30: /MD9 -> /MD7
- DD7 pad 31: /MD10 -> /~MRD
- DD7 pad 32: /MD11 -> /A11
- DD7 pad 33: VCC -> /A9
- DD7 pad 34: GND -> /A10
- DD7 pad 35: /MD12 -> /MA16
- DD7 pad 36: /MD13 -> (no net)
- DD7 pad 9: /MD2 -> VCC
- DD8 pad 1: /MA17 -> /MA18
- DD8 pad 10: /MD3 -> GND
- DD8 pad 11: VCC -> /MD2
- DD8 pad 12: GND -> /MD3
- DD8 pad 13: /MD4 -> /~MWR
- DD8 pad 14: /MD5 -> /A0
- DD8 pad 15: /MD6 -> /A2
- DD8 pad 16: /MD7 -> /A4
- DD8 pad 17: /~MWR -> /A6
- DD8 pad 18: /A0 -> /A12
- DD8 pad 19: /A2 -> (no net)
- DD8 pad 2: /MA16 -> /MA17
- DD8 pad 20: /A4 -> /A7
- DD8 pad 21: /A6 -> /A5
- DD8 pad 22: /A12 -> /A3
- DD8 pad 23: /A7 -> /A1
- DD8 pad 24: /A5 -> /A8
- DD8 pad 25: /A3 -> /MD4
- DD8 pad 26: /A1 -> /MD5
- DD8 pad 27: /A8 -> VCC
- DD8 pad 28: (no net) -> GND
- DD8 pad 29: /MD8 -> /MD6
- DD8 pad 30: /MD9 -> /MD7
- DD8 pad 31: /MD10 -> /~MRD
- DD8 pad 32: /MD11 -> /A11
- DD8 pad 33: VCC -> /A9
- DD8 pad 34: GND -> /A10
- DD8 pad 35: /MD12 -> /MA16
- DD8 pad 36: /MD13 -> (no net)
- DD8 pad 9: /MD2 -> VCC
- DD9 pad 1: /MA17 -> /MA18
- DD9 pad 10: /MD3 -> GND
- DD9 pad 11: VCC -> /MD2
- DD9 pad 12: GND -> /MD3
- DD9 pad 13: /MD4 -> /~MWR
- DD9 pad 14: /MD5 -> /A0
- DD9 pad 15: /MD6 -> /A2
- DD9 pad 16: /MD7 -> /A4
- DD9 pad 17: /~MWR -> /A6
- DD9 pad 18: /A0 -> /A12
- DD9 pad 19: /A2 -> (no net)
- DD9 pad 2: /MA16 -> /MA17
- DD9 pad 20: /A4 -> /A7
- DD9 pad 21: /A6 -> /A5
- DD9 pad 22: /A12 -> /A3
- DD9 pad 23: /A7 -> /A1
- DD9 pad 24: /A5 -> /A8
- DD9 pad 25: /A3 -> /MD4
- DD9 pad 26: /A1 -> /MD5
- DD9 pad 27: /A8 -> VCC
- DD9 pad 28: (no net) -> GND
- DD9 pad 29: /MD8 -> /MD6
- DD9 pad 30: /MD9 -> /MD7
- DD9 pad 31: /MD10 -> /~MRD
- DD9 pad 32: /MD11 -> /A11
- DD9 pad 33: VCC -> /A9
- DD9 pad 34: GND -> /A10
- DD9 pad 35: /MD12 -> /MA16
- DD9 pad 36: /MD13 -> (no net)
- DD9 pad 9: /MD2 -> VCC
- J1 pad 15b: /~LB -> /MA16
- J1 pad 19b: Net-(J1-Pad19b) -> /SND
Routing:
- net GND: track 129.1 -> 1226.9 mm, vias 0 -> 186
- net VCC: track 467.4 -> 912.1 mm, vias 8 -> 29
- net /~LB: track 67.1 -> 0.00 mm, vias 3 -> 0
- net /TCK: track 0.00 -> 62.6 mm
- net /X0: track 0.00 -> 59.8 mm
- net /~UB: track 64.8 -> 7.52 mm, vias 3 -> 0
- net /TDO: track 0.00 -> 56.4 mm, vias 0 -> 2
- net /MA16: track 38.2 -> 93.1 mm
- net /A13: track 56.2 -> 110.6 mm, vias 3 -> 5
- net /TMS: track 0.00 -> 52.3 mm
- net /MD14: track 47.7 -> 0.00 mm, vias 2 -> 0
- net /MD15: track 47.7 -> 0.00 mm, vias 2 -> 0
- net /MD11: track 47.7 -> 0.00 mm, vias 2 -> 0
- net /MD10: track 47.7 -> 0.00 mm, vias 2 -> 0
- net /MD9: track 47.7 -> 0.00 mm, vias 2 -> 0
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Other:
- board text added: "PRO/128 ROM/HDD MENU PGD CP/M-80 MC7007 HDD FDD"
- board text added: "R0"
- board text added: "R1"
- board text added: "R2"

Commit message: RC версия процессорного модуля
Parts:
- added C2-2: TestPoint_Pad_D1.5mm, TestPoint:TestPoint_Pad_D1.5mm, F.Cu at (86.9, 95.2)
- added C23: CP, Capacitors_Tantalum_SMD:CP_Tantalum_Case-A_EIA-3216-18_Hand, B.Cu at (141.0, 135.3)
- added JP1: R16B, Pin_Headers:Pin_Header_Straight_1x02_Pitch2.54mm, F.Cu at (100.6, 85.7)
- added R34: 1K, Resistor_SMD:R_0805_2012Metric, B.Cu at (103.6, 79.9)
- added REF**: TestPoint_Pad_1.0x1.0mm, TestPoint:TestPoint_Pad_1.0x1.0mm, B.Cu at (111.3, 88.1)
- C11, DD6, DD8, R23, R25, R26, R27: moved to B.Cu
- C2, C21, C3, C4, C5, C6, C8, R14: moved to F.Cu
- SW3: footprint Buttons_Switches_ThroughHole:SW_PUSH_6mm -> Button_Switch_THT:SW_Tactile_SPST_Angled_PTS645Vx83-2LFS
- moved DD1 93.5 mm to (83.8, 136.5), turned to 90 degrees
- moved C10 75.5 mm to (149.9, 129.7), turned to 90 degrees
- moved R32 66.4 mm to (130.4, 90.8), turned to 270 degrees
- moved J2 65.4 mm to (130.4, 93.6), turned to 270 degrees
- moved R29 62.7 mm to (125.3, 99.2), turned to 90 degrees
- moved R30 59.5 mm to (125.3, 90.8), turned to 270 degrees
- moved R12 58.5 mm to (150.5, 121.3), turned to 180 degrees
- moved DD3 56.7 mm to (151.1, 118.7), turned to 0 degrees
- moved R10 54.9 mm to (133.3, 114.3)
- moved R11 54.9 mm to (133.3, 111.8)
- moved R9 54.9 mm to (133.3, 116.8)
- moved SW2 54.9 mm to (136.5, 116.8)
- moved R14 52.8 mm to (118.1, 70.6), turned to 180 degrees
- moved R31 52.5 mm to (120.3, 90.8), turned to 270 degrees
- moved C11 52.4 mm to (157.5, 108.8), turned to 90 degrees
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Connections:
- net Net-(DD3-Pad31) renamed /PGM1
- net Net-(DD4-Pad31) renamed /PGM2
- net Net-(DD5-Pad31) renamed /PGM3
- DD10 pad 11: /D7 -> /D0
- DD10 pad 12: /D6 -> /D1
- DD10 pad 13: /D5 -> /D2
- DD10 pad 14: /D4 -> /D3
- DD10 pad 15: /D3 -> /D4
- DD10 pad 16: /D2 -> /D5
- DD10 pad 17: /D1 -> /D6
- DD10 pad 18: /D0 -> /D7
- DD10 pad 2: /MD7 -> /MD3
- DD10 pad 3: /MD0 -> /MD2
- DD10 pad 4: /MD6 -> /MD1
- DD10 pad 5: /MD1 -> /MD0
- DD10 pad 6: /MD2 -> /MD7
- DD10 pad 7: /MD5 -> /MD6
- DD10 pad 8: /MD3 -> /MD5
- DD12 pad 1: /~IRQ0 -> /~IRQS
- DD12 pad 10: /~IRQ7 -> /~IORQ
- DD12 pad 11: /~IRQS -> /~IRQ0
- DD12 pad 14: /D4 -> /~INT
- DD12 pad 15: /D3 -> /D7
- DD12 pad 16: /D5 -> /D6
- DD12 pad 17: /D6 -> /D5
- DD12 pad 18: /~IORQ -> /D4
- DD12 pad 19: /D2 -> /D3
- DD12 pad 2: /~INT -> /~IRQ7
- DD12 pad 20: /D7 -> /D2
- DD12 pad 21: /D0 -> /D1
- DD12 pad 22: /D1 -> /D0
- DD12 pad 3: /~M1 -> /~IRQ6
- DD12 pad 4: /~IRQ1 -> /~IRQ5
- DD12 pad 5: /~IRQ2 -> /~IRQ4
- DD12 pad 7: /~IRQ4 -> /~IRQ2
- DD12 pad 8: /~IRQ5 -> /~IRQ1
- DD12 pad 9: /~IRQ6 -> /~M1
- DD2 pad 1: /MA17 -> /~VCE
- DD2 pad 10: /R2A14 -> /~VO0
- DD2 pad 100: /~VO0 -> /pFA
- DD2 pad 12: /R2A17 -> /~OE0
- DD2 pad 13: /R2A18 -> /~OE1
- DD2 pad 14: /R2A16 -> /~CE0
- DD2 pad 16: /R2A15 -> /~CE1
- DD2 pad 17: /CFG0 -> /~CE2
- DD2 pad 19: /CFG1 -> /~CE3
- DD2 pad 2: /MA18 -> /MA15
- DD2 pad 20: /CFG2 -> /A2
- DD2 pad 21: /CFG3 -> /A14
- DD2 pad 22: /CFG4 -> /~RFSH
- DD2 pad 23: /CFG5 -> /MA14
- DD2 pad 24: /CFG6 -> /A1
- DD2 pad 25: /CFG7 -> /D0
- DD2 pad 27: /~R1 -> /A7
- DD2 pad 28: /~R2 -> /A5
- DD2 pad 29: /~R3 -> /D1
- DD2 pad 30: /~RD -> /A12
- DD2 pad 31: /~IORQ -> /ZA15
- DD2 pad 32: /~WR -> /A4
- DD2 pad 33: /~MREQ -> /~RD
- DD2 pad 35: /~WAIT -> /A15
- DD2 pad 36: /~IRQ0 -> /A13
- DD2 pad 37: /~RES -> /INT50
- DD2 pad 40: /D1 -> /~MRD
- DD2 pad 41: /~M1 -> /~MWR
- DD2 pad 42: /D0 -> /~R1
- DD2 pad 44: /~RFSH -> /R2A13
- DD2 pad 45: /D7 -> /R2A14
- DD2 pad 46: /D6 -> /R2A17
- DD2 pad 47: /D5 -> /R2A15
- DD2 pad 48: /D4 -> /R2A16
- DD2 pad 49: /D3 -> /~R2
- DD2 pad 5: /~CE3 -> /MA18
- DD2 pad 50: /D2 -> /~R3
- DD2 pad 52: /A0 -> /R2A18
- DD2 pad 53: /A1 -> /~IRQ0
- DD2 pad 54: /A2 -> /A0
- DD2 pad 55: /A3 -> /D5
- DD2 pad 56: /A4 -> /A11
- DD2 pad 57: /A5 -> /~BLIO
- DD2 pad 58: /A6 -> /~WAIT
- DD2 pad 6: /~CE2 -> /MA17
- DD2 pad 60: /ZA15 -> /CSL
- DD2 pad 61: /A7 -> /D6
- DD2 pad 63: /ZA14 -> /pFB
- DD2 pad 64: /A8 -> /D7
- DD2 pad 65: /A13 -> /A6
- DD2 pad 67: /A9 -> /D4
- DD2 pad 68: /A12 -> /A9
- DD2 pad 7: /~CE1 -> /MA16
- DD2 pad 70: /A11 -> /CFG0
- DD2 pad 71: /r2 -> /CFG1
- DD2 pad 72: /~TRB -> /CFG2
- DD2 pad 75: /INT50 -> /CFG3
- DD2 pad 76: /SND -> /CFG4
- DD2 pad 77: Net-(DD2-Pad77) -> /CFG5
- DD2 pad 78: /~OE0 -> /CFG6
- DD2 pad 79: /MA14 -> /CFG7
- DD2 pad 8: /~CE0 -> /D2
- DD2 pad 80: /A14 -> /D3
- DD2 pad 81: /MA15 -> /A8
- DD2 pad 83: /A15 -> Net-(DD2-Pad83)
- DD2 pad 84: Net-(DD2-Pad84) -> /ZCLK
- DD2 pad 85: /MA16 -> /ZA14
- DD2 pad 88: /R1 -> /~IORQ
- DD2 pad 89: /~BLIO -> /~RES
- DD2 pad 9: /R2A13 -> /~VO1
- DD2 pad 90: /R0 -> /~WR
- DD2 pad 92: /~VCE -> /~M1
- DD2 pad 93: /~MWR -> /~MREQ
- DD2 pad 94: /~MRD -> /pF8
- DD2 pad 96: /pFA -> /SND
- DD2 pad 97: /pF8 -> /A3
- DD2 pad 98: /pFC -> /R16B
- DD2 pad 99: /~VO1 -> /pFC
- DD3 pad 22: /~R1 -> /~RD
- DD3 pad 24: /~RD -> /~R1
- DD4 pad 22: /~R2 -> /~RD
- DD4 pad 24: /~RD -> /~R2
- DD5 pad 22: /~R3 -> /~RD
- DD5 pad 24: /~RD -> /~R3
- DD6 pad 1: /MA18 -> /A8
- DD6 pad 14: /A0 -> /A7
- DD6 pad 15: /A2 -> /A5
- DD6 pad 16: /A4 -> /A3
- DD6 pad 17: /A6 -> /A1
- DD6 pad 2: /MA17 -> /A13
- DD6 pad 20: /A7 -> /A0
- DD6 pad 21: /A5 -> /A2
- DD6 pad 22: /A3 -> /A4
- DD6 pad 23: /A1 -> /A6
- DD6 pad 24: /A8 -> /MA14
- DD6 pad 3: /MA15 -> /A9
- DD6 pad 32: /A11 -> /MA15
- DD6 pad 33: /A9 -> /MA16
- DD6 pad 34: /A10 -> /MA17
- DD6 pad 35: /MA16 -> /MA18
- DD6 pad 4: /MA14 -> /A10
- DD6 pad 5: /A13 -> /A11
- DD7 pad 1: /MA18 -> /A8
- DD7 pad 14: /A0 -> /A7
- DD7 pad 15: /A2 -> /A5
- DD7 pad 16: /A4 -> /A3
- DD7 pad 17: /A6 -> /A1
- DD7 pad 2: /MA17 -> /A13
- DD7 pad 20: /A7 -> /A0
- DD7 pad 21: /A5 -> /A2
- DD7 pad 22: /A3 -> /A4
- DD7 pad 23: /A1 -> /A6
- DD7 pad 24: /A8 -> /MA14
- DD7 pad 3: /MA15 -> /A9
- DD7 pad 32: /A11 -> /MA15
- DD7 pad 33: /A9 -> /MA16
- DD7 pad 34: /A10 -> /MA17
- DD7 pad 35: /MA16 -> /MA18
- DD7 pad 4: /MA14 -> /A10
- DD7 pad 5: /A13 -> /A11
- DD8 pad 1: /MA18 -> /A8
- DD8 pad 14: /A0 -> /A7
- DD8 pad 15: /A2 -> /A5
- DD8 pad 16: /A4 -> /A3
- DD8 pad 17: /A6 -> /A1
- DD8 pad 2: /MA17 -> /A13
- DD8 pad 20: /A7 -> /A0
- DD8 pad 21: /A5 -> /A2
- DD8 pad 22: /A3 -> /A4
- DD8 pad 23: /A1 -> /A6
- DD8 pad 24: /A8 -> /MA14
- DD8 pad 3: /MA15 -> /A9
- DD8 pad 32: /A11 -> /MA15
- DD8 pad 33: /A9 -> /MA16
- DD8 pad 34: /A10 -> /MA17
- DD8 pad 35: /MA16 -> /MA18
- DD8 pad 4: /MA14 -> /A10
- DD8 pad 5: /A13 -> /A11
- DD9 pad 1: /MA18 -> /A8
- DD9 pad 14: /A0 -> /A7
- DD9 pad 15: /A2 -> /A5
- DD9 pad 16: /A4 -> /A3
- DD9 pad 17: /A6 -> /A1
- DD9 pad 2: /MA17 -> /A13
- DD9 pad 20: /A7 -> /A0
- DD9 pad 21: /A5 -> /A2
- DD9 pad 22: /A3 -> /A4
- DD9 pad 23: /A1 -> /A6
- DD9 pad 24: /A8 -> /MA14
- DD9 pad 3: /MA15 -> /A9
- DD9 pad 32: /A11 -> /MA15
- DD9 pad 33: /A9 -> /MA16
- DD9 pad 34: /A10 -> /MA17
- DD9 pad 35: /MA16 -> /MA18
- DD9 pad 4: /MA14 -> /A10
- DD9 pad 5: /A13 -> /A11
- J1 pad 31b: /~TRB -> Net-(J1-Pad31b)
- J1 pad 32b: /ZCLK -> Net-(J1-Pad32b)
- R10 pad 2: /R1A13 -> /R1A14
- R11 pad 2: /R1A14 -> /R1A13
- SW2 pad 2: /R1A13 -> /R1A14
- SW2 pad 3: /R1A14 -> /R1A13
- SW3 pad 1: Net-(SW3-Pad1) -> GND
- SW3 pad 2: Net-(SW3-Pad2) -> /~RES
Routing:
- net GND: track 1226.9 -> 1522.7 mm, vias 186 -> 198
- net /~RES: track 143.0 -> 277.8 mm
- net /INT50: track 43.4 -> 127.2 mm, vias 1 -> 4
- net /A12: track 259.8 -> 329.3 mm, vias 7 -> 9
- net /~INT: track 29.8 -> 99.2 mm, vias 0 -> 4
- net /~IRQ1: track 75.8 -> 11.5 mm
- net /MA14: track 86.5 -> 148.8 mm
- net /~IRQ2: track 71.1 -> 11.5 mm
- net VCC: track 912.1 -> 969.0 mm, vias 29 -> 30
- net /~IRQ3: track 66.4 -> 11.5 mm
- net /A14: track 19.2 -> 73.6 mm, vias 0 -> 2
- net /~MWR: track 95.3 -> 149.3 mm, vias 3 -> 5
- net /~IRQ4: track 61.7 -> 11.5 mm
- net /A11: track 207.2 -> 256.6 mm, vias 6 -> 5
- net /~RD: track 218.0 -> 168.7 mm, vias 4 -> 6
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Other:
- net class Default: clearance 0.175 -> 0.176
- rule trace_clearance: 0.175 -> 0.176
- rule trace_min: 0.16 -> 0.17
- board text removed: "R0"
- board text removed: "R1"
- board text removed: "R2"

Commit message: Обновлена плата процессорного модуля - версия для производства.
Parts:
- removed C2-2: TestPoint_Pad_D1.5mm, TestPoint:TestPoint_Pad_D1.5mm
- removed C21: 100n, Capacitor_SMD:C_0805_2012Metric
- removed DD10: AP6, Package_SO:SOIC-20W_7.5x12.8mm_P1.27mm
- added R35: 1K, Resistor_SMD:R_0805_2012Metric, F.Cu at (122.6, 104.4)
- moved C2 0.64 mm to (93.0, 94.4)
- moved C3 0.64 mm to (86.5, 101.6)
- moved DD6 0.63 mm to (81.9, 63.4)
- moved DD7 0.63 mm to (81.9, 78.7)
- moved DD8 0.63 mm to (81.9, 93.9)
- moved DD9 0.63 mm to (81.9, 109.2)
Connections:
- DD6 pad 11: /MD2 -> /D4
- DD6 pad 12: /MD3 -> /D6
- DD6 pad 25: /MD4 -> /D7
- DD6 pad 26: /MD5 -> /D5
- DD6 pad 29: /MD6 -> /D2
- DD6 pad 30: /MD7 -> /D0
- DD6 pad 4: /A10 -> /A11
- DD6 pad 5: /A11 -> /A10
- DD6 pad 7: /MD0 -> /D1
- DD6 pad 8: /MD1 -> /D3
- DD7 pad 11: /MD2 -> /D4
- DD7 pad 12: /MD3 -> /D6
- DD7 pad 25: /MD4 -> /D7
- DD7 pad 26: /MD5 -> /D5
- DD7 pad 29: /MD6 -> /D2
- DD7 pad 30: /MD7 -> /D0
- DD7 pad 4: /A10 -> /A11
- DD7 pad 5: /A11 -> /A10
- DD7 pad 7: /MD0 -> /D1
- DD7 pad 8: /MD1 -> /D3
- DD8 pad 11: /MD2 -> /D4
- DD8 pad 12: /MD3 -> /D6
- DD8 pad 25: /MD4 -> /D7
- DD8 pad 26: /MD5 -> /D5
- DD8 pad 29: /MD6 -> /D2
- DD8 pad 30: /MD7 -> /D0
- DD8 pad 4: /A10 -> /A11
- DD8 pad 5: /A11 -> /A10
- DD8 pad 7: /MD0 -> /D1
- DD8 pad 8: /MD1 -> /D3
- DD9 pad 11: /MD2 -> /D4
- DD9 pad 12: /MD3 -> /D6
- DD9 pad 25: /MD4 -> /D7
- DD9 pad 26: /MD5 -> /D5
- DD9 pad 29: /MD6 -> /D2
- DD9 pad 30: /MD7 -> /D0
- DD9 pad 4: /A10 -> /A11
- DD9 pad 5: /A11 -> /A10
- DD9 pad 7: /MD0 -> /D1
- DD9 pad 8: /MD1 -> /D3
Routing:
- net GND: track 1522.7 -> 1373.9 mm, vias 198 -> 176
- net /MD3: track 69.9 -> 0.00 mm, vias 2 -> 0
- net /MD2: track 68.9 -> 0.00 mm, vias 2 -> 0
- net /MD4: track 67.1 -> 0.00 mm, vias 2 -> 0
- net /MD5: track 66.5 -> 0.00 mm, vias 2 -> 0
- net /MD1: track 65.4 -> 0.00 mm, vias 2 -> 0
- net /MD0: track 64.5 -> 0.00 mm, vias 2 -> 0
- net /D1: track 221.1 -> 285.1 mm, vias 3 -> 4
- net /MD6: track 61.8 -> 0.00 mm, vias 2 -> 0
- net /MD7: track 59.7 -> 0.00 mm, vias 2 -> 0
- net /D2: track 251.3 -> 307.3 mm, vias 6 -> 7
- net /D7: track 203.8 -> 258.0 mm, vias 6 -> 7
- net /D6: track 218.5 -> 264.8 mm, vias 6 -> 7
- net /D5: track 230.2 -> 274.7 mm, vias 6 -> 7
- net /~OE0: track 45.5 -> 2.67 mm, vias 3 -> 1
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