File: hardware/orion_cpu/orion_cpu.sch (KiCad schematic (older format))
At the start: 47 parts, among them J1 C96ABC, SW1 CONFIG, SW2 ROM1

Commit message: Обновлён проект платы процессорного модуля
Parts:
- removed DD11: AP6, Package_SO:SOIC-20W_7.5x12.8mm_P1.27mm, symbol orion:AP6
- removed DD6, DD7, DD8, DD9: AS7C4098A, Projects:SOJ-44, symbol orion:AS7C4098A
- added C21, C22: 100n, Capacitor_SMD:C_0805_2012Metric, symbol Device:C
- added DD11: 74AHCT1G04, Package_TO_SOT_SMD:SOT-353_SC-70-5_Handsoldering, symbol 74xGxx:74AHCT1G04
- added DD6, DD7, DD8, DD9: CY7C1049B, Projects:SOJ-36, symbol orion:CY7C1049B
- added J2: JTAG, Connector_PinHeader_2.54mm:PinHeader_2x05_P2.54mm_Vertical, symbol Connector:AVR-JTAG-10
- added R13, R14, R15, R16, R17, R18, R19, R20, R21, R22, R23, R24, R25, R26, R27, R28, R29, R30, R31, R32, R33: 1K, Resistor_SMD:R_0805_2012Metric, symbol Device:R
- added SW3: RESET, Buttons_Switches_ThroughHole:SW_PUSH_6mm, symbol Switch:SW_Push
Connections:
- net labels added: MA18, R0, R1, VDD, r2
- net labels removed: MD10, MD11, MD12, MD13, MD14, MD15, MD8, MD9, PGM1, PGM2, R2, R3, pFB, ~LB
- wire segments 639 -> 672
- no-connect marks 24 -> 25
Other:
- moved on the sheet: C13, C14, C15, C16, C17, C18, C19, C20

Commit message: RC версия процессорного модуля
Parts:
- added C23: CP, Capacitors_Tantalum_SMD:CP_Tantalum_Case-A_EIA-3216-18_Hand, symbol Device:CP
- added JP1: R16B, Pin_Headers:Pin_Header_Straight_1x02_Pitch2.54mm, symbol Device:Jumper
- added R34: 1K, Resistor_SMD:R_0805_2012Metric, symbol Device:R
- SW3: footprint Buttons_Switches_ThroughHole:SW_PUSH_6mm -> Button_Switch_THT:SW_Tactile_SPST_Angled_PTS645Vx83-2LFS
Connections:
- net R0 is gone; now on net ~WR: DD2.90 (I/OE2/GCLK2)
- net R1 is gone; now on net ~IORQ: DD2.88 (I/OE1)
- net r2 is gone; now on net CFG1: DD2.71 (IO)
- net A0: now also DD2.54 (IO), DD6.20 (A10), DD7.20 (A10), DD8.20 (A10), DD9.20 (A10); no longer DD2.52 (IO), DD6.14 (A5), DD7.14 (A5), DD8.14 (A5), DD9.14 (A5)
- net A1: now also DD2.24 (IO), DD6.17 (A8), DD7.17 (A8), DD8.17 (A8), DD9.17 (A8); no longer DD2.53 (IO), DD6.23 (A13), DD7.23 (A13), DD8.23 (A13), DD9.23 (A13)
- net A10: now also DD6.4 (A3), DD7.4 (A3), DD8.4 (A3), DD9.4 (A3); no longer DD6.34 (A17), DD7.34 (A17), DD8.34 (A17), DD9.34 (A17)
- net A11: now also DD2.56 (IO), DD6.5 (A4), DD7.5 (A4), DD8.5 (A4), DD9.5 (A4); no longer DD2.70 (IO), DD6.32 (A15), DD7.32 (A15), DD8.32 (A15), DD9.32 (A15)
- net A12: now also DD2.30 (IO); no longer DD2.68 (IO)
- net A13: now also DD2.36 (IO), DD6.2 (A1), DD7.2 (A1), DD8.2 (A1), DD9.2 (A1); no longer DD2.65 (IO), DD6.5 (A4), DD7.5 (A4), DD8.5 (A4), DD9.5 (A4)
- net A14: now also DD2.21 (IO); no longer DD2.80 (IO)
- net A15: now also DD2.35 (IO); no longer DD2.83 (IO)
- net A2: now also DD2.20 (IO), DD6.21 (A11), DD7.21 (A11), DD8.21 (A11), DD9.21 (A11); no longer DD2.54 (IO), DD6.15 (A6), DD7.15 (A6), DD8.15 (A6), DD9.15 (A6)
- net A3: now also DD2.97 (IO), DD6.16 (A7), DD7.16 (A7), DD8.16 (A7), DD9.16 (A7); no longer DD2.55 (IO), DD6.22 (A12), DD7.22 (A12), DD8.22 (A12), DD9.22 (A12)
- net A4: now also DD2.32 (IO), DD6.22 (A12), DD7.22 (A12), DD8.22 (A12), DD9.22 (A12); no longer DD2.56 (IO), DD6.16 (A7), DD7.16 (A7), DD8.16 (A7), DD9.16 (A7)
- net A5: now also DD2.28 (IO), DD6.15 (A6), DD7.15 (A6), DD8.15 (A6), DD9.15 (A6); no longer DD2.57 (IO), DD6.21 (A11), DD7.21 (A11), DD8.21 (A11), DD9.21 (A11)
- net A6: now also DD2.65 (IO), DD6.23 (A13), DD7.23 (A13), DD8.23 (A13), DD9.23 (A13); no longer DD2.58 (IO), DD6.17 (A8), DD7.17 (A8), DD8.17 (A8), DD9.17 (A8)
- net A7: now also DD2.27 (IO), DD6.14 (A5), DD7.14 (A5), DD8.14 (A5), DD9.14 (A5); no longer DD2.61 (O), DD6.20 (A10), DD7.20 (A10), DD8.20 (A10), DD9.20 (A10)
- net A8: now also DD2.81 (IO), DD6.1 (A0), DD7.1 (A0), DD8.1 (A0), DD9.1 (A0); no longer DD2.64 (IO), DD6.24 (A14), DD7.24 (A14), DD8.24 (A14), DD9.24 (A14)
- net A9: now also DD2.68 (IO), DD6.3 (A2), DD7.3 (A2), DD8.3 (A2), DD9.3 (A2); no longer DD2.67 (IO), DD6.33 (A16), DD7.33 (A16), DD8.33 (A16), DD9.33 (A16)
- net CFG0: now also DD2.70 (IO); no longer DD2.17 (IO)
- net CFG1: no longer DD2.19 (IO)
- net CFG2: now also DD2.72 (IO); no longer DD2.20 (IO)
- net CFG3: now also DD2.75 (IO); no longer DD2.21 (IO)
- net CFG4: now also DD2.76 (IO); no longer DD2.22 (IO)
- net CFG5: now also DD2.77 (IO); no longer DD2.23 (IO)
- net CFG6: now also DD2.78 (IO); no longer DD2.24 (IO)
- net CFG7: now also DD2.79 (IO); no longer DD2.25 (IO)
- net D0: now also DD10.11 (B7), DD12.22 (IO2), DD2.25 (IO); no longer DD10.18 (B0), DD12.21 (IO3), DD2.42 (IO)
- net D1: now also DD10.12 (B6), DD12.21 (IO3), DD2.29 (IO); no longer DD10.17 (B1), DD12.22 (IO2), DD2.40 (IO)
- net D2: now also DD10.13 (B5), DD12.20 (IO4), DD2.8 (IO); no longer DD10.16 (B2), DD12.19 (IO5), DD2.50 (IO)
- net D3: now also DD10.14 (B4), DD12.19 (IO5), DD2.80 (IO); no longer DD10.15 (B3), DD12.15 (IO9), DD2.49 (IO)
- net D4: now also DD10.15 (B3), DD12.18 (IO6), DD2.67 (IO); no longer DD10.14 (B4), DD12.14 (IO10), DD2.48 (IO)
- net D5: now also DD10.16 (B2), DD12.17 (IO7), DD2.55 (IO); no longer DD10.13 (B5), DD12.16 (IO8), DD2.47 (IO)
- net D6: now also DD10.17 (B1), DD12.16 (IO8), DD2.61 (O); no longer DD10.12 (B6), DD12.17 (IO7), DD2.46 (IO)
- net D7: now also DD10.18 (B0), DD12.15 (IO9), DD2.64 (IO); no longer DD10.11 (B7), DD12.20 (IO4), DD2.45 (IO)
- net GND: now also SW3.1, C23.2, JP1.2
- net INT50: now also DD2.37 (IO); no longer DD2.75 (IO)
- net MA14: now also DD2.23 (IO), DD6.24 (A14), DD7.24 (A14), DD8.24 (A14), DD9.24 (A14); no longer DD2.79 (IO), DD6.4 (A3), DD7.4 (A3), DD8.4 (A3), DD9.4 (A3)
- net MA15: now also DD2.2 (IO), DD6.32 (A15), DD7.32 (A15), DD8.32 (A15), DD9.32 (A15); no longer DD2.81 (IO), DD6.3 (A2), DD7.3 (A2), DD8.3 (A2), DD9.3 (A2)
- net MA16: now also DD2.7 (IO), DD6.33 (A16), DD7.33 (A16), DD8.33 (A16), DD9.33 (A16); no longer DD2.85 (IO), DD6.35 (A18), DD7.35 (A18), DD8.35 (A18), DD9.35 (A18)
- net MA17: now also DD2.6 (IO), DD6.34 (A17), DD7.34 (A17), DD8.34 (A17), DD9.34 (A17); no longer DD2.1 (IO), DD6.2 (A1), DD7.2 (A1), DD8.2 (A1), DD9.2 (A1)
- net MA18: now also DD2.5 (IO), DD6.35 (A18), DD7.35 (A18), DD8.35 (A18), DD9.35 (A18); no longer DD2.2 (IO), DD6.1 (A0), DD7.1 (A0), DD8.1 (A0), DD9.1 (A0)
- net MD0: now also DD10.5 (A3); no longer DD10.3 (A1)
- net MD1: now also DD10.4 (A2); no longer DD10.5 (A3)
- net MD2: now also DD10.3 (A1); no longer DD10.6 (A4)
- net MD3: now also DD10.2 (A0); no longer DD10.8 (A6)
- net MD5: now also DD10.8 (A6); no longer DD10.7 (A5)
- net MD6: now also DD10.7 (A5); no longer DD10.4 (A2)
- net MD7: now also DD10.6 (A4); no longer DD10.2 (A0)
- net R1A13: now also R11.2, SW2.3; no longer R10.2, SW2.2
- net R1A14: now also R10.2, SW2.2; no longer R11.2, SW2.3
- net R2A13: now also DD2.44 (IO); no longer DD2.9 (IO)
- net R2A14: now also DD2.45 (IO); no longer DD2.10 (IO)
- net R2A15: now also DD2.47 (IO); no longer DD2.16 (IO)
- net R2A16: now also DD2.48 (IO); no longer DD2.14 (IO)
- net R2A17: now also DD2.46 (IO); no longer DD2.12 (IO)
- net R2A18: now also DD2.52 (IO); no longer DD2.13 (IO)
- net SND: now also DD2.96 (IO); no longer DD2.76 (IO)
- net VCC: now also R34.1
- net ZA14: now also DD2.85 (IO); no longer DD2.63 (IO)
- net ZA15: now also DD2.31 (IO); no longer DD2.60 (IO)
- net ZCLK: now also DD2.84 (IO); no longer J1.32b (32B)
- net pF8: now also DD2.94 (IO); no longer DD2.97 (IO)
- net pFA: now also DD2.100 (IO); no longer DD2.96 (IO)
- net pFC: now also DD2.99 (IO); no longer DD2.98 (IO)
- net ~BLIO: now also DD2.57 (IO); no longer DD2.89 (I/GCLR)
- net ~CE0: now also DD2.14 (IO); no longer DD2.8 (IO)
- net ~CE1: now also DD2.16 (IO); no longer DD2.7 (IO)
- net ~CE2: now also DD2.17 (IO); no longer DD2.6 (IO)
- net ~CE3: now also DD2.19 (IO); no longer DD2.5 (IO)
- net ~INT: now also DD12.14 (IO10); no longer DD12.2 (I2)
- net ~IORQ: now also DD12.10 (I10); no longer DD12.18 (IO6), DD2.31 (IO)
- net ~IRQ0: now also DD12.11 (I11), DD2.53 (IO); no longer DD12.1 (I1/CLK), DD2.36 (IO)
- net ~IRQ1: now also DD12.8 (I8); no longer DD12.4 (I4)
- net ~IRQ2: now also DD12.7 (I7); no longer DD12.5 (I5)
- net ~IRQ4: now also DD12.5 (I5); no longer DD12.7 (I7)
- net ~IRQ5: now also DD12.4 (I4); no longer DD12.8 (I8)
- net ~IRQ6: now also DD12.3 (I3); no longer DD12.9 (I9)
- net ~IRQ7: now also DD12.2 (I2); no longer DD12.10 (I10)
- net ~IRQS: now also DD12.1 (I1/CLK); no longer DD12.11 (I11)
- net ~M1: now also DD12.9 (I9), DD2.92 (IO); no longer DD12.3 (I3), DD2.41 (IO)
- net ~MRD: now also DD2.40 (IO); no longer DD2.94 (IO)
- net ~MREQ: now also DD2.93 (IO); no longer DD2.33 (IO)
- net ~MWR: now also DD2.41 (IO); no longer DD2.93 (IO)
- net ~OE0: now also DD2.12 (IO); no longer DD2.78 (IO)
- net ~OE1: now also DD2.13 (IO)
- net ~R1: now also DD2.42 (IO), DD3.24 (OE); no longer DD2.27 (IO), DD3.22 (CE)
- net ~R2: now also DD2.49 (IO), DD4.24 (OE); no longer DD2.28 (IO), DD4.22 (CE)
- net ~R3: now also DD2.50 (IO), DD5.24 (OE); no longer DD2.29 (IO), DD5.22 (CE)
- net ~RD: now also DD2.33 (IO), DD3.22 (CE), DD4.22 (CE), DD5.22 (CE); no longer DD2.30 (IO), DD3.24 (OE), DD4.24 (OE), DD5.24 (OE)
- net ~RES: now also DD2.89 (I/GCLR), SW3.2, C23.1; no longer DD2.37 (IO)
- net ~RFSH: now also DD2.22 (IO); no longer DD2.44 (IO)
- net ~VCE: now also DD2.1 (IO); no longer DD2.92 (IO)
- net ~VO0: now also DD2.10 (IO); no longer DD2.100 (IO)
- net ~VO1: now also DD2.9 (IO); no longer DD2.99 (IO)
- net ~WAIT: now also DD2.58 (IO); no longer DD2.35 (IO)
- net ~WR: no longer DD2.32 (IO)
- net PGM2: now reaches DD4.31 (PGM), R28.2
- net PGM3: now reaches DD5.31 (PGM), R33.2
- net PGM1: now reaches DD3.31 (PGM), R12.2
- net ~TRB: no longer names the net of J1.31b (31B)
- net ~TRB: no longer DD2.72 (IO)
- new net CSL: DD2.60 (IO)
- new net R16B: DD2.98 (IO), JP1.1, R34.2
- new net pFB: DD2.63 (IO)
- no-connect marks 25 -> 27
Other:
- moved on the sheet: C13, C14, C15, C16, C17, C18, C19, C20, C21, C22, DD10, DD11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

Commit message: Обновлена плата процессорного модуля - версия для производства.
Parts:
- added JP2: CSL, Pin_Headers:Pin_Header_Straight_1x02_Pitch2.54mm, symbol Device:Jumper
- added R35: 1K, Resistor_SMD:R_0805_2012Metric, symbol Device:R
Connections:
- net A10: now also DD6.5 (A4), DD7.5 (A4), DD8.5 (A4), DD9.5 (A4); no longer DD6.4 (A3), DD7.4 (A3), DD8.4 (A3), DD9.4 (A3)
- net A11: now also DD6.4 (A3), DD7.4 (A3), DD8.4 (A3), DD9.4 (A3); no longer DD6.5 (A4), DD7.5 (A4), DD8.5 (A4), DD9.5 (A4)
- net CSL: now also JP2.1, R35.2
- net D0: now also DD6.30 (Q7), DD7.30 (Q7), DD8.30 (Q7), DD9.30 (Q7); no longer DD10.11 (B7)
- net D1: now also DD6.7 (Q0), DD7.7 (Q0), DD8.7 (Q0), DD9.7 (Q0); no longer DD10.12 (B6)
- net D2: now also DD6.29 (Q6), DD7.29 (Q6), DD8.29 (Q6), DD9.29 (Q6); no longer DD10.13 (B5)
- net D3: now also DD6.8 (Q1), DD7.8 (Q1), DD8.8 (Q1), DD9.8 (Q1); no longer DD10.14 (B4)
- net D4: now also DD6.11 (Q2), DD7.11 (Q2), DD8.11 (Q2), DD9.11 (Q2); no longer DD10.15 (B3)
- net D5: now also DD6.26 (Q5), DD7.26 (Q5), DD8.26 (Q5), DD9.26 (Q5); no longer DD10.16 (B2)
- net D6: now also DD6.12 (Q3), DD7.12 (Q3), DD8.12 (Q3), DD9.12 (Q3); no longer DD10.17 (B1)
- net D7: now also DD6.25 (Q4), DD7.25 (Q4), DD8.25 (Q4), DD9.25 (Q4); no longer DD10.18 (B0)
- net GND: now also JP2.2
- net VCC: now also R35.1
- net ~MWR: no longer DD10.1 (A>B)
- net ~OE0: no longer DD10.19 (OE)
- removed net MD0: DD10.5 (A3), DD6.7 (Q0), DD7.7 (Q0), DD8.7 (Q0), DD9.7 (Q0)
- removed net MD1: DD10.4 (A2), DD6.8 (Q1), DD7.8 (Q1), DD8.8 (Q1), DD9.8 (Q1)
- removed net MD2: DD10.3 (A1), DD6.11 (Q2), DD7.11 (Q2), DD8.11 (Q2), DD9.11 (Q2)
- removed net MD3: DD10.2 (A0), DD6.12 (Q3), DD7.12 (Q3), DD8.12 (Q3), DD9.12 (Q3)
- removed net MD4: DD10.9 (A7), DD6.25 (Q4), DD7.25 (Q4), DD8.25 (Q4), DD9.25 (Q4)
- removed net MD5: DD10.8 (A6), DD6.26 (Q5), DD7.26 (Q5), DD8.26 (Q5), DD9.26 (Q5)
- removed net MD6: DD10.7 (A5), DD6.29 (Q6), DD7.29 (Q6), DD8.29 (Q6), DD9.29 (Q6)
- removed net MD7: DD10.6 (A4), DD6.30 (Q7), DD7.30 (Q7), DD8.30 (Q7), DD9.30 (Q7)
