File: hardware/orion_video/orion_video.kicad_pcb (KiCad board)
At the start: 2 copper layers, 99.7 x 99.7 mm, 74 parts, among them J1 C96ABC, J2 VGA, J3 VGAP, J4 4:3, J5 10/5, Y1 25MHz

Commit message: Актуализированна аппаратная часть
Parts:
- removed R10: 1k, Resistor_SMD:R_0805_2012Metric
- removed R12: 470, Resistor_SMD:R_0805_2012Metric
- removed R9: 510, Resistor_SMD:R_0805_2012Metric
- removed REF** (x2): MountingHole_3.2mm_M3_Pad, Mounting_Holes:MountingHole_3.2mm_M3_Pad
- removed Y1: 25MHz, Crystal:Crystal_SMD_7050-4Pin_7.0x5.0mm
- added C21: 100n, Capacitor_SMD:C_0805_2012Metric, F.Cu at (89.5, 103.5)
- added C22: 100n, Capacitor_SMD:C_0805_2012Metric, F.Cu at (65.4, 114.9)
- added C23: 100n, Capacitor_SMD:C_0805_2012Metric, F.Cu at (101.1, 73.0)
- added C24: 100n, Capacitor_SMD:C_0805_2012Metric, F.Cu at (87.5, 67.7)
- added C25: 100n, Capacitor_SMD:C_0805_2012Metric, B.Cu at (73.8, 67.9)
- added C26: 100n, Capacitor_SMD:C_0805_2012Metric, B.Cu at (73.0, 97.2)
- added C27: 100n, Capacitor_SMD:C_0805_2012Metric, F.Cu at (88.0, 97.2)
- added C28: 100n, Capacitor_SMD:C_0805_2012Metric, F.Cu at (108.7, 76.5)
- added C29: 100n, Capacitor_SMD:C_0805_2012Metric, F.Cu at (150.5, 122.9)
- added CPX1: TestPoint_Small, TestPoint:TestPoint_THTPad_D1.0mm_Drill0.5mm, F.Cu at (114.9, 111.0)
- added DD26: IR23, Package_SO:SOIC-20W_7.5x12.8mm_P1.27mm, B.Cu at (80.6, 93.3)
- added DD27: 74AHC1G04, Package_TO_SOT_SMD:SOT-23-5, F.Cu at (87.0, 84.5)
- added DD28: Conn_02x08_Counter_Clockwise, Package_SO:SOIC-16_3.9x9.9mm_P1.27mm, F.Cu at (127.8, 131.4)
- added DD29: Conn_02x10_Counter_Clockwise, Package_SO:SOIC-20W_7.5x12.8mm_P1.27mm, F.Cu at (143.6, 130.3)
- added F85: FA2, TestPoint:TestPoint_THTPad_D1.0mm_Drill0.5mm, B.Cu at (72.4, 75.8)
- added F86: FA2, TestPoint:TestPoint_THTPad_D1.0mm_Drill0.5mm, B.Cu at (72.4, 74.0)
- added F87: FA2, TestPoint:TestPoint_THTPad_D1.0mm_Drill0.5mm, B.Cu at (89.2, 74.3)
- added FA2: FA2, TestPoint:TestPoint_THTPad_D1.0mm_Drill0.5mm, B.Cu at (88.3, 70.1)
- added FA3: FA3, TestPoint:TestPoint_THTPad_D1.0mm_Drill0.5mm, B.Cu at (73.7, 70.5)
- added FA4: FA4, TestPoint:TestPoint_THTPad_D1.0mm_Drill0.5mm, B.Cu at (73.7, 79.4)
- added FA5: FA5, TestPoint:TestPoint_THTPad_D1.0mm_Drill0.5mm, B.Cu at (73.9, 76.8)
- added FA6: FA6, TestPoint:TestPoint_THTPad_D1.0mm_Drill0.5mm, B.Cu at (73.9, 73.0)
- added GL19: GL14, TestPoint:TestPoint_THTPad_D1.0mm_Drill0.5mm, F.Cu at (125.1, 111.0)
- added GL20: GL15, TestPoint:TestPoint_THTPad_D1.0mm_Drill0.5mm, F.Cu at (122.6, 111.0)
- added GL21: GL16, TestPoint:TestPoint_THTPad_D1.0mm_Drill0.5mm, F.Cu at (120.0, 111.0)
- added GL22: GL22, TestPoint:TestPoint_THTPad_D1.0mm_Drill0.5mm, F.Cu at (117.5, 111.0)
- added GX18: GX18, TestPoint:TestPoint_THTPad_D1.0mm_Drill0.5mm, B.Cu at (151.1, 86.4)
- added GX19: GX19, TestPoint:TestPoint_THTPad_D1.0mm_Drill0.5mm, B.Cu at (148.6, 86.4)
- added GX20: GX20, TestPoint:TestPoint_THTPad_D1.0mm_Drill0.5mm, B.Cu at (146.1, 86.4)
- added GY15: GY15, TestPoint:TestPoint_THTPad_D1.0mm_Drill0.5mm, B.Cu at (141.0, 83.8)
- added GY16: GY16, TestPoint:TestPoint_THTPad_D1.0mm_Drill0.5mm, B.Cu at (143.5, 83.8)
- added GY17: GY17, TestPoint:TestPoint_THTPad_D1.0mm_Drill0.5mm, B.Cu at (146.1, 83.8)
- added GY18: GY22, TestPoint:TestPoint_THTPad_D1.0mm_Drill0.5mm, B.Cu at (148.6, 83.8)
- added H1: MountingHole, MountingHole:MountingHole_3.2mm_M3, F.Cu at (163.8, 134.6)
- added H2: MountingHole, MountingHole:MountingHole_3.2mm_M3, F.Cu at (74.3, 134.6)
- added H3: MountingHole, MountingHole:MountingHole_2mm, F.Cu at (50.2, 132.1)
- added H4: MountingHole, MountingHole:MountingHole_2mm, F.Cu at (57.0, 131.4)
- added H5: MountingHole, MountingHole:MountingHole_2mm, F.Cu at (57.0, 125.9)
- added H6: MountingHole, MountingHole:MountingHole_2mm, F.Cu at (51.4, 125.9)
- added J6: Conn_01x09_Female, Connector_PinHeader_1.27mm:PinHeader_1x09_P1.27mm_Vertical, F.Cu at (151.1, 125.9)
- added PS0: TestPoint_Small, TestPoint:TestPoint_THTPad_D1.0mm_Drill0.5mm, F.Cu at (85.1, 105.4)
- added PS1: TestPoint_Small, TestPoint:TestPoint_THTPad_D1.0mm_Drill0.5mm, F.Cu at (83.8, 106.7)
- added PS2: TestPoint_Small, TestPoint:TestPoint_THTPad_D1.0mm_Drill0.5mm, F.Cu at (81.3, 106.7)
- added PS3: TestPoint_Small, TestPoint:TestPoint_THTPad_D1.0mm_Drill0.5mm, F.Cu at (80.0, 105.4)
- added PS4: TestPoint_Small, TestPoint:TestPoint_THTPad_D1.0mm_Drill0.5mm, F.Cu at (76.2, 106.7)
- added PS5: TestPoint_Small, TestPoint:TestPoint_THTPad_D1.0mm_Drill0.5mm, F.Cu at (77.5, 105.4)
- added PS6: TestPoint_Small, TestPoint:TestPoint_THTPad_D1.0mm_Drill0.5mm, F.Cu at (78.7, 106.7)
- added PS7: TestPoint_Small, TestPoint:TestPoint_THTPad_D1.0mm_Drill0.5mm, F.Cu at (82.5, 105.4)
- added R22: 470, Resistor_SMD:R_0805_2012Metric, F.Cu at (90.3, 128.7)
- added R23: 1K, Resistor_SMD:R_0805_2012Metric, F.Cu at (91.4, 123.8)
- added R24: 510, Resistor_SMD:R_0805_2012Metric, F.Cu at (88.9, 123.8)
- added R25: 47, Resistor_SMD:R_0805_2012Metric, F.Cu at (119.0, 136.1)
- added R26: 47, Resistor_SMD:R_0805_2012Metric, F.Cu at (114.8, 137.7)
- added SW1: SW_DIP_04, Button_Switch_THT:SW_DIP_SPSTx04_Slide_9.78x12.34mm_W7.62mm_P2.54mm, F.Cu at (155.6, 128.3)
- added TP1: SW2, TestPoint:TestPoint_THTPad_D1.0mm_Drill0.5mm, F.Cu at (158.1, 118.1)
- added TP2: SW3, TestPoint:TestPoint_THTPad_D1.0mm_Drill0.5mm, F.Cu at (155.6, 118.1)
- added TP3: GL13, TestPoint:TestPoint_THTPad_D1.0mm_Drill0.5mm, F.Cu at (132.7, 122.7)
- added VD0: TestPoint_Small, TestPoint:TestPoint_THTPad_D1.0mm_Drill0.5mm, B.Cu at (106.7, 86.4)
- added VD1: TestPoint_Small, TestPoint:TestPoint_THTPad_D1.0mm_Drill0.5mm, B.Cu at (108.0, 85.1)
- added VD10: TestPoint_Small, TestPoint:TestPoint_THTPad_D1.0mm_Drill0.5mm, B.Cu at (95.2, 85.1)
- added VD11: TestPoint_Small, TestPoint:TestPoint_THTPad_D1.0mm_Drill0.5mm, B.Cu at (96.5, 86.4)
- added VD12: TestPoint_Small, TestPoint:TestPoint_THTPad_D1.0mm_Drill0.5mm, B.Cu at (100.3, 85.1)
- added VD13: TestPoint_Small, TestPoint:TestPoint_THTPad_D1.0mm_Drill0.5mm, B.Cu at (99.1, 86.4)
- added VD14: TestPoint_Small, TestPoint:TestPoint_THTPad_D1.0mm_Drill0.5mm, B.Cu at (97.8, 85.1)
- added VD15: TestPoint_Small, TestPoint:TestPoint_THTPad_D1.0mm_Drill0.5mm, B.Cu at (94.0, 86.4)
- added VD2: TestPoint_Small, TestPoint:TestPoint_THTPad_D1.0mm_Drill0.5mm, B.Cu at (110.5, 85.1)
- added VD3: TestPoint_Small, TestPoint:TestPoint_THTPad_D1.0mm_Drill0.5mm, B.Cu at (111.8, 86.4)
- added VD4: TestPoint_Small, TestPoint:TestPoint_THTPad_D1.0mm_Drill0.5mm, B.Cu at (115.6, 85.1)
- added VD5: TestPoint_Small, TestPoint:TestPoint_THTPad_D1.0mm_Drill0.5mm, B.Cu at (114.3, 86.4)
- added VD6: TestPoint_Small, TestPoint:TestPoint_THTPad_D1.0mm_Drill0.5mm, B.Cu at (113.0, 85.1)
- added VD7: TestPoint_Small, TestPoint:TestPoint_THTPad_D1.0mm_Drill0.5mm, B.Cu at (109.2, 86.4)
- added VD8: TestPoint_Small, TestPoint:TestPoint_THTPad_D1.0mm_Drill0.5mm, B.Cu at (91.4, 86.4)
- added VD9: TestPoint_Small, TestPoint:TestPoint_THTPad_D1.0mm_Drill0.5mm, B.Cu at (92.7, 85.1)
- added X1: 50MHz, Crystal:Crystal_SMD_7050-4Pin_7.0x5.0mm, F.Cu at (114.4, 127.9)
- added ~BL1: Jumper_NC_Small, Connector_PinHeader_2.00mm:PinHeader_1x02_P2.00mm_Vertical, F.Cu at (107.3, 113.6)
- C1, C10, C11, C12, C13, C16, C17, C2, C20, C3, C4, C6, C7, C8: moved to F.Cu
- DD1: value IE18 -> TM2; footprint Package_SO:SOIC-16_3.9x9.9mm_P1.27mm -> Package_SO:SOIC-14_3.9x8.7mm_P1.27mm
- DD10: value IR33 -> IE18; footprint Package_SO:SOIC-20W_7.5x12.8mm_P1.27mm -> Package_SO:SOIC-16_3.9x9.9mm_P1.27mm
- DD11: value IR33 -> ATF22V10; footprint Package_SO:SOIC-20W_7.5x12.8mm_P1.27mm -> Package_DIP:DIP-24_W7.62mm
- DD12: value IR33 -> IDT7028PF; footprint Package_SO:SOIC-20W_7.5x12.8mm_P1.27mm -> Package_QFP:LQFP-100_14x14mm_P0.5mm; moved to F.Cu
- DD14: value IR10 -> IR33; footprint Package_SO:SOIC-16_3.9x9.9mm_P1.27mm -> Package_SO:SOIC-20W_7.5x12.8mm_P1.27mm; moved to B.Cu
- DD15: value IR10 -> IR33; footprint Package_SO:SOIC-16_3.9x9.9mm_P1.27mm -> Package_SO:SOIC-20W_7.5x12.8mm_P1.27mm
- DD16: value IR10 -> IR33; footprint Package_SO:SOIC-16_3.9x9.9mm_P1.27mm -> Package_SO:SOIC-20W_7.5x12.8mm_P1.27mm; moved to F.Cu
- DD18: value ATF22V10 -> IR10; footprint Package_DIP:DIP-24_W7.62mm -> Package_SO:SOIC-16_3.9x9.9mm_P1.27mm; moved to B.Cu
- DD19: value AP6 -> IR10; footprint Package_SO:SOIC-20W_7.5x12.8mm_P1.27mm -> Package_SO:SOIC-16_3.9x9.9mm_P1.27mm
- DD2, DD7: value IE18 -> ATF22V10; footprint Package_SO:SOIC-16_3.9x9.9mm_P1.27mm -> Package_DIP:DIP-24_W7.62mm
- DD20: value AP6 -> IR10; footprint Package_SO:SOIC-20W_7.5x12.8mm_P1.27mm -> Package_SO:SOIC-16_3.9x9.9mm_P1.27mm; moved to F.Cu
- DD21: value TM9 -> ATF22V10; footprint Package_SO:SOIC-16_3.9x9.9mm_P1.27mm -> Package_DIP:DIP-24_W7.62mm
- DD22: value TM9 -> AP6; footprint Package_SO:SOIC-16_3.9x9.9mm_P1.27mm -> Package_SO:SOIC-20W_7.5x12.8mm_P1.27mm; moved to F.Cu
- DD23: value 74AHCT1G04 -> IR35; footprint Package_TO_SOT_SMD:SOT-353_SC-70-5_Handsoldering -> Package_SO:SOIC-20W_7.5x12.8mm_P1.27mm
- DD24: value IR23 -> IR35; moved to B.Cu
- DD25: value IR23 -> 6; moved to F.Cu
- DD4, DD8: value ATF22V10 -> IE18; footprint Package_DIP:DIP-24_W7.62mm -> Package_SO:SOIC-16_3.9x9.9mm_P1.27mm
- DD6: value IE18 -> 74AHCT1GU04; footprint Package_SO:SOIC-16_3.9x9.9mm_P1.27mm -> Package_TO_SOT_SMD:SOT-23-5
- DD9: value IDT7028PF -> IE18; footprint Package_QFP:LQFP-100_14x14mm_P0.5mm -> Package_SO:SOIC-16_3.9x9.9mm_P1.27mm
- J1: footprint Connectors_IEC_DIN:Socket_DIN41612-CaseC1-full-Male-96Pin-3rows -> orion:Socket_DIN41612-CaseC1-full-Male-96Pin-3rows
- J2: footprint w_conn_pc:DB_15F-VGA -> Connector_Dsub:DSUB-15-HD_Female_Horizontal_P2.29x1.98mm_EdgePinOffset3.03mm_Housed_MountingHolesOffset4.94mm
- J3: value VGAP -> Conn_01x07_Female; footprint Connector_PinHeader_2.54mm:PinHeader_1x03_P2.54mm_Vertical -> Connector_PinHeader_1.27mm:PinHeader_1x07_P1.27mm_Vertical
- J4: value 4:3 -> Conn_01x07_Female; footprint Connector_PinHeader_2.54mm:PinHeader_1x02_P2.54mm_Vertical -> Connector_PinHeader_1.27mm:PinHeader_1x07_P1.27mm_Vertical
- J5: value 10/5 -> Conn_01x09_Female; footprint Connector_PinHeader_2.54mm:PinHeader_1x02_P2.54mm_Vertical -> Connector_PinHeader_1.27mm:PinHeader_1x09_P1.27mm_Vertical
- R1, R2, R3: value 1k -> 1K; moved to F.Cu
- R11: value 510 -> 1k
- R15: value 470 -> 1K
- R16: value 470 -> 510
- R18: value 47 -> 470
- R19: value 47 -> 1K
- R20: value 1k -> 510
- R21: value 1k -> 470
- R4, R5, R6: value 1k -> 1K
- R7: value 510 -> 1K
- moved R21 69.2 mm to (91.6, 126.6), turned to 180 degrees
- moved R7 68.3 mm to (166.2, 66.2), turned to 90 degrees
- moved R20 67.4 mm to (94.0, 123.8), turned to -90 degrees
- moved R5 63.4 mm to (59.1, 86.2), turned to 180 degrees
- moved R8 62.6 mm to (119.0, 58.5), turned to 0 degrees
- moved DD11 58.3 mm to (163.8, 73.7)
- moved R3 54.2 mm to (158.1, 115.6), turned to -90 degrees
- moved R18 53.8 mm to (95.4, 128.7), turned to 180 degrees
- moved C11 53.2 mm to (166.4, 80.3), turned to 90 degrees
- moved DD10 52.2 mm to (137.2, 66.0)
- moved R2 51.9 mm to (160.7, 115.6), turned to -90 degrees
- moved C16 51.3 mm to (117.3, 101.1)
- moved R19 49.9 mm to (96.5, 123.8), turned to -90 degrees
- moved C13 48.4 mm to (117.1, 56.6), turned to 180 degrees
- moved R4 47.5 mm to (155.6, 115.6), turned to -90 degrees
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Connections:
- net /VL24 renamed VL0
- net /VL26 renamed VL2
- net /VL28 renamed VL4
- net /VL29 renamed VL5
- DD1 pad 1: /~XRES -> Net-(DD1-Pad1)
- DD1 pad 10: Net-(DD1-Pad10) -> Net-(DD1-Pad1)
- DD1 pad 11: /X3 -> /FEND
- DD1 pad 12: /X2 -> /VB0
- DD1 pad 13: /X1 -> Net-(DD1-Pad1)
- DD1 pad 14: /X0 -> VCC
- DD1 pad 2: /CLK -> /VB1
- DD1 pad 3: Net-(DD1-Pad3) -> /FEND
- DD1 pad 4: Net-(DD1-Pad4) -> Net-(DD1-Pad1)
- DD1 pad 5: Net-(DD1-Pad5) -> (no net)
- DD1 pad 7: Net-(DD1-Pad10) -> GND
- DD1 pad 8: GND -> Net-(DD1-Pad8)
- DD1 pad 9: Net-(DD1-Pad10) -> (no net)
- DD10 pad 1: GND -> /video_gen/~YRES
- DD10 pad 10: GND -> /video_gen/YH1
- DD10 pad 11: /CL0 -> (no net)
- DD10 pad 12: /VL0 -> (no net)
- DD10 pad 13: /VL7 -> /video_gen/Y9
- DD10 pad 14: /VL1 -> /video_gen/Y8
- DD10 pad 15: /VL2 -> (no net)
- DD10 pad 16: /VL6 -> VCC
- DD10 pad 2: /VD4 -> Net-(DD10-Pad2)
- DD10 pad 3: /VD5 -> (no net)
- DD10 pad 4: /VD3 -> (no net)
- DD10 pad 5: /VD6 -> (no net)
- DD10 pad 6: /VD2 -> (no net)
- DD10 pad 7: /VD1 -> Net-(DD10-Pad7)
- DD10 pad 8: /VD7 -> GND
- DD10 pad 9: /VD0 -> Net-(DD10-Pad7)
- DD11 pad 1: GND -> /video_gen/XLE
- DD11 pad 10: GND -> /video_gen/Y8
- DD11 pad 11: /CL0 -> /video_gen/Y9
- DD11 pad 12: /VL8 -> GND
- DD11 pad 13: /VL15 -> /video_gen/SR0
- DD11 pad 14: /VL9 -> /video_gen/SR1
- DD11 pad 15: /VL10 -> Net-(DD11-Pad15)
- DD11 pad 16: /VL14 -> Net-(DD11-Pad16)
- DD11 pad 17: /VL11 -> Net-(DD11-Pad17)
- DD11 pad 18: /VL13 -> Net-(DD11-Pad18)
- DD11 pad 19: /VL12 -> /VS
- DD11 pad 2: /VD12 -> /video_gen/Y0
- DD11 pad 20: VCC -> /video_gen/~BV
- DD11 pad 3: /VD13 -> /video_gen/Y1
- DD11 pad 4: /VD11 -> /video_gen/Y2
- DD11 pad 5: /VD14 -> /video_gen/Y3
- DD11 pad 6: /VD10 -> /video_gen/Y4
- DD11 pad 7: /VD9 -> /video_gen/Y5
- DD11 pad 8: /VD15 -> /video_gen/Y6
- DD11 pad 9: /VD8 -> /video_gen/Y7
- DD12 pad 1: GND -> /video_regs/A9
- DD12 pad 10: GND -> /video_regs/~UB
- DD12 pad 11: /CL1 -> /video_regs/MA16
- DD12 pad 12: /VL20 -> /video_regs/~VCE
- DD12 pad 13: /VL21 -> MVP
- DD12 pad 14: /VL19 -> MVP
- DD12 pad 15: /VL22 -> VCC
- DD12 pad 16: /VL18 -> /video_regs/~MWR
- DD12 pad 17: /VL17 -> /video_regs/~MRD
- DD12 pad 18: /VL23 -> GND
- DD12 pad 19: /VL16 -> GND
- DD12 pad 2: /VD0 -> /video_regs/A10
- DD12 pad 20: VCC -> /video_regs/BD4
- DD12 pad 3: /VD7 -> /video_regs/A11
- DD12 pad 4: /VD1 -> /video_regs/A12
- DD12 pad 5: /VD2 -> /video_regs/A13
- DD12 pad 6: /VD6 -> /video_regs/MA14
- DD12 pad 7: /VD3 -> /video_regs/MA15
- DD12 pad 8: /VD5 -> (no net)
- DD12 pad 9: /VD4 -> (no net)
- DD13 pad 11: /CL1 -> /CL0
- DD13 pad 14: /VL27 -> VL6
- DD13 pad 15: /VL30 -> VL3
- DD13 pad 17: /VL25 -> VL7
- DD13 pad 18: /VL31 -> VL1
- DD13 pad 2: /VD8 -> /VD0
- DD13 pad 3: /VD15 -> /VD1
- DD13 pad 4: /VD9 -> /VD7
- DD13 pad 5: /VD10 -> /VD2
- DD13 pad 6: /VD14 -> /VD3
- DD13 pad 7: /VD11 -> /VD6
- DD13 pad 8: /VD13 -> /VD5
- DD13 pad 9: /VD12 -> /VD4
- DD14 pad 1: Net-(DD14-Pad1) -> GND
- DD14 pad 10: /VL4 -> GND
- DD14 pad 11: /VL5 -> /CL0
- DD14 pad 12: /VL6 -> VL12
- DD14 pad 13: /P0 -> VL13
- DD14 pad 14: /VL7 -> VL14
- DD14 pad 15: /~BE -> VL11
- DD14 pad 16: VCC -> VL10
- DD14 pad 2: /VL0 -> /VD8
- DD14 pad 3: /VL1 -> /VD9
- DD14 pad 4: /VL2 -> /VD15
- DD14 pad 5: /VL3 -> /VD10
- DD14 pad 6: GND -> /VD11
- DD14 pad 7: /CLK -> /VD14
- DD14 pad 8: GND -> /VD13
- DD14 pad 9: PUP1 -> /VD12
- DD15 pad 1: Net-(DD15-Pad1) -> GND
- DD15 pad 10: /VL12 -> GND
- DD15 pad 11: /VL13 -> /CL1
- DD15 pad 12: /VL14 -> VL16
- DD15 pad 13: /P1 -> VL17
- DD15 pad 14: /VL15 -> VL23
- DD15 pad 15: /~BE -> VL18
- DD15 pad 16: VCC -> VL19
- DD15 pad 2: /VL8 -> /VD4
- DD15 pad 3: /VL9 -> /VD5
- DD15 pad 4: /VL10 -> /VD6
- DD15 pad 5: /VL11 -> /VD3
- DD15 pad 6: GND -> /VD2
- DD15 pad 7: /CLK -> /VD7
- DD15 pad 8: GND -> /VD1
- DD15 pad 9: /VM2 -> /VD0
- DD16 pad 1: Net-(DD16-Pad1) -> GND
- DD16 pad 10: /VL20 -> GND
- DD16 pad 11: /VL21 -> /CL1
- DD16 pad 12: /VL22 -> VL24
- DD16 pad 13: /P2 -> VL25
- DD16 pad 14: /VL23 -> VL31
- DD16 pad 15: /~BE -> VL26
- DD16 pad 16: VCC -> VL27
- DD16 pad 2: /VL16 -> /VD12
- DD16 pad 3: /VL17 -> /VD13
- DD16 pad 4: /VL18 -> /VD14
- DD16 pad 5: /VL19 -> /VD11
- DD16 pad 6: GND -> /VD10
- DD16 pad 7: /CLK -> /VD15
- DD16 pad 8: GND -> /VD9
- DD16 pad 9: PUP1 -> /VD8
- DD17 pad 12: /VL30 -> VL6
- DD17 pad 13: /P3 -> /video_regs/P0
- DD17 pad 14: /VL31 -> VL7
- DD17 pad 3: /VL25 -> VL1
- DD17 pad 5: /VL27 -> VL3
- DD17 pad 7: /CLK -> /CPX
- DD17 pad 9: PUP1 -> Net-(DD17-Pad1)
- DD18 pad 1: /~BL -> Net-(DD17-Pad1)
- DD18 pad 10: /PS1 -> VL12
- DD18 pad 11: /PS0 -> VL13
- DD18 pad 12: GND -> VL14
- DD18 pad 13: /PS7 -> /video_regs/P1
- DD18 pad 14: /PS6 -> VL15
- DD18 pad 15: /PS5 -> /~BE
- DD18 pad 16: /PS4 -> VCC
- DD18 pad 2: /P3 -> VL8
- DD18 pad 3: /P1 -> VL9
- DD18 pad 4: /VM1 -> VL10
- DD18 pad 5: /VM0 -> VL11
- DD18 pad 6: /VM4 -> GND
- DD18 pad 7: /P0 -> /CPX
- DD18 pad 8: /PS3 -> GND
- DD18 pad 9: /PS2 -> /VM2
- DD19 pad 1: /~MWR -> Net-(DD17-Pad1)
- DD19 pad 10: GND -> VL20
- DD19 pad 11: /D4 -> VL21
- DD19 pad 12: /D5 -> VL22
- DD19 pad 13: /D3 -> /video_regs/P2
- DD19 pad 14: /D6 -> VL23
- DD19 pad 15: /D2 -> /~BE
- DD19 pad 16: /D1 -> VCC
- DD19 pad 2: /MD0 -> VL16
- DD19 pad 3: /MD7 -> VL17
- DD19 pad 4: /MD1 -> VL18
- DD19 pad 5: /MD2 -> VL19
- DD19 pad 6: /MD6 -> GND
- DD19 pad 7: /MD3 -> /CPX
- DD19 pad 8: /MD5 -> GND
- DD19 pad 9: /MD4 -> Net-(DD17-Pad1)
- DD2 pad 1: /~XRES -> Net-(DD2-Pad1)
- DD2 pad 10: /XH0 -> /CL1
- DD2 pad 11: /X7 -> /video_gen/SR0
- DD2 pad 12: /X6 -> GND
- DD2 pad 13: /X5 -> /video_gen/SR1
- DD2 pad 14: /X4 -> Net-(DD12-Pad70)
- DD2 pad 15: /XH1 -> Net-(DD12-Pad69)
- DD2 pad 16: VCC -> /VS2
- DD2 pad 2: /CLK -> Net-(DD1-Pad8)
- DD2 pad 3: Net-(DD2-Pad3) -> Net-(DD1-Pad6)
- DD2 pad 4: Net-(DD2-Pad4) -> /VM3
- DD2 pad 5: Net-(DD2-Pad5) -> /VM2
- DD2 pad 6: Net-(DD2-Pad6) -> /VM0
- DD2 pad 7: Net-(DD1-Pad10) -> /VM1
- DD2 pad 8: GND -> /VM4
- DD2 pad 9: Net-(DD1-Pad10) -> Net-(DD2-Pad9)
- DD20 pad 1: /~MWR -> Net-(DD17-Pad1)
- DD20 pad 10: GND -> VL28
- DD20 pad 11: /D0 -> VL29
- DD20 pad 12: /D7 -> VL30
- DD20 pad 13: /D1 -> /video_regs/P3
- DD20 pad 14: /D2 -> VL31
- DD20 pad 15: /D6 -> /~BE
- DD20 pad 16: /D3 -> VCC
- DD20 pad 2: /MD12 -> VL24
- DD20 pad 3: /MD13 -> VL25
- DD20 pad 4: /MD11 -> VL26
- DD20 pad 5: /MD14 -> VL27
- DD20 pad 6: /MD10 -> GND
- DD20 pad 7: /MD9 -> /CPX
- DD20 pad 8: /MD15 -> GND
- DD20 pad 9: /MD8 -> Net-(DD17-Pad1)
- DD21 pad 1: /~RES -> /video_regs/P2
- DD21 pad 10: /VB1 -> /video_regs/PS3
- DD21 pad 11: /D1 -> /video_regs/PS5
- DD21 pad 12: /F1 -> GND
- DD21 pad 13: /D3 -> /video_regs/PS4
- DD21 pad 14: /D7 -> /video_regs/PS6
- DD21 pad 15: /SR16 -> /video_regs/PS2
- DD21 pad 16: VCC -> /video_regs/PS1
- DD21 pad 2: /PGD -> /video_regs/P0
- DD21 pad 3: /D6 -> /~BL
- DD21 pad 4: /D2 -> /video_regs/P3
- DD21 pad 5: /F0 -> /video_regs/P1
- DD21 pad 6: /D0 -> /VS1
- DD21 pad 7: /VB0 -> /VS0
- DD21 pad 8: GND -> /video_regs/PS0
- DD21 pad 9: /PFA -> /video_regs/PS7
- DD22 pad 1: /~RES -> /video_regs/~RD
- DD22 pad 10: /VM0 -> GND
- DD22 pad 11: /D0 -> /video_regs/BD7
- DD22 pad 12: /VM2 -> /video_regs/BD6
- DD22 pad 13: /D2 -> /video_regs/BD5
- DD22 pad 14: Net-(DD22-Pad14) -> /video_regs/BD4
- DD22 pad 15: Net-(DD22-Pad15) -> /video_regs/BD3
- DD22 pad 16: VCC -> /video_regs/BD2
- DD22 pad 2: /VM4 -> /video_regs/D0
- DD22 pad 3: /D4 -> /video_regs/D1
- DD22 pad 4: /D3 -> /video_regs/D2
- DD22 pad 5: /VM3 -> /video_regs/D3
- DD22 pad 6: /D1 -> /video_regs/D4
- DD22 pad 7: /VM1 -> /video_regs/D5
- DD22 pad 8: GND -> /video_regs/D6
- DD22 pad 9: /PF8 -> /video_regs/D7
- DD23 pad 1: (no net) -> /video_regs/~RES
- DD23 pad 2: /VM3 -> Net-(DD23-Pad2)
- DD23 pad 3: GND -> /video_regs/BD3
- DD23 pad 4: /~VM3 -> /video_regs/BD6
- DD23 pad 5: VCC -> Net-(DD23-Pad5)
- DD24 pad 1: /~VM3 -> /video_regs/~RES
- DD24 pad 11: /PFC -> /video_regs/PF8
- DD24 pad 12: /PS7 -> /VM4
- DD24 pad 13: /PS6 -> /video_regs/BD4
- DD24 pad 14: /PS5 -> /video_regs/BD5
- DD24 pad 15: /PS4 -> Net-(DD24-Pad15)
- DD24 pad 16: /PS3 -> Net-(DD24-Pad16)
- DD24 pad 17: /PS2 -> /video_regs/BD6
- DD24 pad 18: /PS1 -> /video_regs/BD3
- DD24 pad 19: /PS0 -> /VM3
- DD24 pad 2: /D0 -> /VM2
- DD24 pad 3: /D1 -> /video_regs/BD2
- DD24 pad 4: /D2 -> /video_regs/BD7
- DD24 pad 5: /D3 -> Net-(DD24-Pad5)
- DD24 pad 6: /D4 -> /VM1
- DD24 pad 7: /D5 -> /video_regs/BD1
- DD24 pad 8: /D6 -> /video_regs/BD0
- DD24 pad 9: /D7 -> /VM0
- DD25 pad 1: /VM3 -> Net-(DD25-Pad1)
- DD25 pad 11: /~BE -> /video_regs/PFC
- DD25 pad 12: /PS0 -> /video_regs/PS4
- DD25 pad 13: /PS1 -> /video_regs/PS5
- DD25 pad 14: /PS2 -> /video_regs/PS6
- DD25 pad 15: /PS3 -> /video_regs/PS3
- DD25 pad 16: /PS4 -> /video_regs/PS2
- DD25 pad 17: /PS5 -> /video_regs/PS7
- DD25 pad 18: /PS6 -> /video_regs/PS1
- DD25 pad 19: /PS7 -> /video_regs/PS0
- DD25 pad 2: /VD15 -> /video_regs/BD0
- DD25 pad 3: /VD14 -> /video_regs/BD1
- DD25 pad 4: /VD13 -> /video_regs/BD7
- DD25 pad 5: /VD12 -> /video_regs/BD2
- DD25 pad 6: /VD11 -> /video_regs/BD3
- DD25 pad 7: /VD10 -> /video_regs/BD6
- DD25 pad 8: /VD9 -> /video_regs/BD5
- DD25 pad 9: /VD8 -> /video_regs/BD4
- DD3 pad 1: /~XRES -> /video_gen/~XRES
- DD3 pad 10: /XH1 -> Net-(DD3-Pad10)
- DD3 pad 11: Net-(DD3-Pad11) -> /video_gen/X3
- DD3 pad 12: Net-(DD3-Pad12) -> /CL1
- DD3 pad 13: /X9 -> /video_gen/X1
- DD3 pad 14: /X8 -> /video_gen/X0
- DD3 pad 15: Net-(DD3-Pad15) -> /video_gen/XH0
- DD3 pad 2: /CLK -> /CPX
- DD3 pad 3: Net-(DD3-Pad3) -> (no net)
- DD3 pad 4: Net-(DD3-Pad4) -> (no net)
- DD3 pad 5: Net-(DD3-Pad5) -> (no net)
- DD3 pad 6: Net-(DD3-Pad6) -> (no net)
- DD3 pad 7: Net-(DD1-Pad10) -> Net-(DD3-Pad10)
- DD3 pad 9: Net-(DD1-Pad10) -> Net-(DD3-Pad10)
- DD4 pad 1: /X0 -> /video_gen/~XRES
- DD4 pad 10: /X9 -> /video_gen/XH0
- DD4 pad 11: /WEN -> /video_gen/X7
- DD4 pad 12: GND -> /video_gen/X6
- DD4 pad 13: /SR16 -> /video_gen/X5
- DD4 pad 14: /ZCLK -> /video_gen/X4
- DD4 pad 15: /~TRB -> /video_gen/XH1
- DD4 pad 16: /CSL -> VCC
- DD4 pad 2: /X1 -> /CPX
- DD4 pad 3: /X2 -> (no net)
- DD4 pad 4: /X3 -> (no net)
- DD4 pad 5: /X4 -> (no net)
- DD4 pad 6: /X5 -> (no net)
- DD4 pad 7: /X6 -> Net-(DD3-Pad10)
- DD4 pad 8: /X7 -> GND
- DD4 pad 9: /X8 -> Net-(DD3-Pad10)
- DD5 pad 1: /~YRES -> /video_gen/~XRES
- DD5 pad 10: Net-(DD5-Pad10) -> /video_gen/XH1
- DD5 pad 11: /Y3 -> (no net)
- DD5 pad 12: /Y2 -> (no net)
- DD5 pad 13: /Y1 -> /video_gen/X9
- DD5 pad 14: /Y0 -> /video_gen/X8
- DD5 pad 15: /YH0 -> (no net)
- DD5 pad 2: /XLE -> /CPX
- DD5 pad 3: Net-(DD5-Pad3) -> (no net)
- DD5 pad 4: Net-(DD5-Pad4) -> (no net)
- DD5 pad 5: Net-(DD5-Pad5) -> (no net)
- DD5 pad 6: Net-(DD5-Pad6) -> (no net)
- DD5 pad 7: Net-(DD5-Pad10) -> Net-(DD3-Pad10)
- DD5 pad 9: Net-(DD5-Pad10) -> Net-(DD3-Pad10)
- DD6 pad 1: /~YRES -> (no net)
- DD6 pad 2: /XLE -> /CL1
- DD6 pad 3: Net-(DD6-Pad3) -> GND
- DD6 pad 4: Net-(DD6-Pad4) -> /CL0
- DD6 pad 5: Net-(DD6-Pad5) -> VCC
- DD7 pad 1: /~YRES -> /video_gen/X0
- DD7 pad 10: /YH1 -> /video_gen/X9
- DD7 pad 11: Net-(DD7-Pad11) -> /video_gen/SR0
- DD7 pad 12: Net-(DD7-Pad12) -> GND
- DD7 pad 13: /Y9 -> /video_gen/SR1
- DD7 pad 14: /Y8 -> /video_gen/XLE
- DD7 pad 15: Net-(DD7-Pad15) -> /video_gen/~XRES
- DD7 pad 16: VCC -> /video_gen/~BV
- DD7 pad 2: /XLE -> /video_gen/X1
- DD7 pad 3: Net-(DD7-Pad3) -> /CL1
- DD7 pad 4: Net-(DD7-Pad4) -> /video_gen/X3
- DD7 pad 5: Net-(DD7-Pad5) -> /video_gen/X4
- DD7 pad 6: Net-(DD7-Pad6) -> /video_gen/X5
- DD7 pad 7: Net-(DD5-Pad10) -> /video_gen/X6
- DD7 pad 8: GND -> /video_gen/X7
- DD7 pad 9: Net-(DD5-Pad10) -> /video_gen/X8
- DD8 pad 1: /Y9 -> /video_gen/~YRES
- DD8 pad 10: /Y0 -> Net-(DD10-Pad7)
- DD8 pad 11: /WEN -> /video_gen/Y3
- DD8 pad 12: GND -> /video_gen/Y2
- DD8 pad 13: /VM4 -> /video_gen/Y1
- DD8 pad 14: /INT50 -> /video_gen/Y0
- DD8 pad 15: /BH -> /video_gen/YH0
- DD8 pad 16: /~BL -> VCC
- DD8 pad 2: /Y8 -> Net-(DD10-Pad2)
- DD8 pad 3: /Y7 -> (no net)
- DD8 pad 4: /Y6 -> (no net)
- DD8 pad 5: /Y5 -> (no net)
- DD8 pad 6: /Y4 -> (no net)
- DD8 pad 7: /Y3 -> Net-(DD10-Pad7)
- DD8 pad 8: /Y2 -> GND
- DD8 pad 9: /Y1 -> Net-(DD10-Pad7)
- DD9 pad 1: /A9 -> /video_gen/~YRES
- DD9 pad 10: /~LB -> /video_gen/YH0
- DD9 pad 11: /~UB -> /video_gen/Y7
- DD9 pad 12: /~VCE0 -> /video_gen/Y6
- DD9 pad 13: PUP3 -> /video_gen/Y5
- DD9 pad 14: PUP3 -> /video_gen/Y4
- DD9 pad 15: VCC -> /video_gen/YH1
- DD9 pad 16: /~MWR -> VCC
- DD9 pad 2: /A10 -> Net-(DD10-Pad2)
- DD9 pad 3: /A11 -> (no net)
- DD9 pad 4: /A12 -> (no net)
- DD9 pad 5: /A13 -> (no net)
- DD9 pad 6: /MA14 -> (no net)
- DD9 pad 7: /MA15 -> Net-(DD10-Pad7)
- DD9 pad 8: (no net) -> GND
- DD9 pad 9: (no net) -> Net-(DD10-Pad7)
- J1 pad 10a: /~WAIT -> (no net)
- J1 pad 10b: Net-(J1-Pad10b) -> (no net)
- J1 pad 10c: /~BLIO -> (no net)
- J1 pad 11a: Net-(J1-Pad11a) -> (no net)
- J1 pad 11b: /~MRD -> /video_regs/~MRD
- J1 pad 11c: /~IORQ -> (no net)
- J1 pad 12a: Net-(J1-Pad12a) -> (no net)
- J1 pad 12b: /~MWR -> /video_regs/~MWR
- J1 pad 12c: /~MREQ -> (no net)
- J1 pad 13a: Net-(J1-Pad13a) -> (no net)
- J1 pad 13b: /~VCE0 -> /video_regs/~VCE
- J1 pad 13c: /~WR -> (no net)
- J1 pad 14a: Net-(J1-Pad14a) -> (no net)
- J1 pad 14b: /~UB -> /video_regs/~UB
- J1 pad 14c: /~RD -> /video_regs/~RD
- J1 pad 15a: Net-(J1-Pad15a) -> (no net)
- J1 pad 15b: /~LB -> /video_regs/MA16
- J1 pad 15c: /HOLD -> (no net)
- J1 pad 16a: /A15 -> (no net)
- J1 pad 16b: /MA15 -> /video_regs/MA15
- J1 pad 17a: /A14 -> (no net)
- J1 pad 17b: /MA14 -> /video_regs/MA14
- J1 pad 17c: /X1 -> (no net)
- J1 pad 18a: /A13 -> /video_regs/A13
- J1 pad 19a: /A12 -> /video_regs/A12
- J1 pad 19b: Net-(J1-Pad19b) -> (no net)
- J1 pad 19c: /~RFSH -> (no net)
- J1 pad 20a: /A11 -> /video_regs/A11
- J1 pad 21a: /A10 -> /video_regs/A10
- J1 pad 21b: Net-(J1-Pad21b) -> (no net)
- J1 pad 21c: /~IRQ1 -> (no net)
- J1 pad 22a: /A9 -> /video_regs/A9
- J1 pad 22b: Net-(J1-Pad22b) -> (no net)
- J1 pad 22c: /~IRQ2 -> (no net)
- J1 pad 23a: /A8 -> /video_regs/A8
- J1 pad 23b: Net-(J1-Pad23b) -> (no net)
- J1 pad 23c: /~IRQ3 -> (no net)
- J1 pad 24a: /A7 -> /video_regs/A7
- J1 pad 24b: Net-(J1-Pad24b) -> (no net)
- J1 pad 24c: /~IRQ4 -> (no net)
- J1 pad 25a: /A6 -> /video_regs/A6
- J1 pad 25b: Net-(J1-Pad25b) -> (no net)
- J1 pad 25c: /~IRQ5 -> (no net)
- J1 pad 26a: /A5 -> /video_regs/A5
- J1 pad 26b: Net-(J1-Pad26b) -> (no net)
- J1 pad 26c: /~IRQ6 -> (no net)
- J1 pad 27a: /A4 -> /video_regs/A4
- J1 pad 27b: Net-(J1-Pad27b) -> (no net)
- J1 pad 27c: /~IRQ7 -> (no net)
- J1 pad 28a: /A3 -> /video_regs/A3
- J1 pad 28b: Net-(J1-Pad28b) -> (no net)
- J1 pad 28c: /~IRQS -> (no net)
- J1 pad 29a: /A2 -> /video_regs/A2
- J1 pad 2a: /D7 -> /video_regs/D7
- J1 pad 2b: Net-(J1-Pad2b) -> (no net)
- J1 pad 2c: /~RES -> /video_regs/~RES
- J1 pad 30a: /A1 -> /video_regs/A1
- J1 pad 30b: /INT50 -> /FEND
- J1 pad 30c: /X0 -> (no net)
- J1 pad 31a: /A0 -> /video_regs/A0
- J1 pad 31b: /~TRB -> (no net)
- J1 pad 32a: /HLDA -> (no net)
- J1 pad 32b: /ZCLK -> (no net)
- J1 pad 3a: /D6 -> /video_regs/D6
- J1 pad 4a: /D5 -> /video_regs/D5
- J1 pad 4b: /~MVO1 -> (no net)
- J1 pad 4c: /~INTA -> (no net)
- J1 pad 5a: /D4 -> /video_regs/D4
- J1 pad 5b: /~MVO0 -> (no net)
- J1 pad 5c: Net-(J1-Pad5c) -> (no net)
- J1 pad 6a: /D3 -> /video_regs/D3
- J1 pad 6b: /PFC -> /video_regs/PFC
- J1 pad 6c: /~M1 -> (no net)
- J1 pad 7a: /D2 -> /video_regs/D2
- J1 pad 7b: /PF8 -> /video_regs/PF8
- J1 pad 7c: Net-(J1-Pad7c) -> (no net)
- J1 pad 8a: /D1 -> /video_regs/D1
- J1 pad 8b: /PFA -> /video_regs/PFA
- J1 pad 8c: /~BLRAM -> (no net)
- J1 pad 9a: /D0 -> /video_regs/D0
- J1 pad 9b: Net-(J1-Pad9b) -> (no net)
- J1 pad 9c: Net-(J1-Pad9c) -> (no net)
- J2 pad 1: /VR -> Net-(J2-Pad1)
- J2 pad 11: Net-(J2-Pad11) -> (no net)
- J2 pad 12: Net-(J2-Pad12) -> (no net)
- J2 pad 15: Net-(J2-Pad15) -> (no net)
- J2 pad 2: /VG -> Net-(J2-Pad2)
- J2 pad 3: /VB -> Net-(J2-Pad3)
- J2 pad 4: Net-(J2-Pad4) -> (no net)
- J2 pad 9: VGAP -> (no net)
- J3 pad 1: GND -> Net-(DD28-Pad1)
- J3 pad 2: VGAP -> Net-(DD28-Pad2)
- J3 pad 3: VCC -> Net-(DD28-Pad3)
- J4 pad 1: GND -> Net-(DD28-Pad15)
- J4 pad 2: /WEN -> Net-(DD28-Pad14)
- J5 pad 1: GND -> Net-(DD29-Pad1)
- J5 pad 2: /CSL -> Net-(DD29-Pad2)
- R1 pad 2: Net-(DD1-Pad10) -> /video_gen/SR0
- R11 pad 1: /VB -> VCC
- R11 pad 2: /IB -> Net-(DD17-Pad1)
- R13 pad 1: Net-(R12-Pad2) -> GND
- R13 pad 2: /VR -> Net-(R13-Pad2)
- R14 pad 1: GND -> Net-(R13-Pad2)
- R14 pad 2: Net-(R14-Pad2) -> Net-(J2-Pad1)
- R15 pad 1: Net-(R14-Pad2) -> Net-(DD21-Pad23)
- R15 pad 2: /VG -> Net-(R13-Pad2)
- R16 pad 1: GND -> Net-(DD21-Pad22)
- R16 pad 2: Net-(R10-Pad1) -> Net-(J2-Pad1)
- R17 pad 1: Net-(R10-Pad1) -> GND
- R17 pad 2: /VB -> Net-(R17-Pad2)
- R18 pad 1: Net-(J2-Pad13) -> Net-(R17-Pad2)
- R18 pad 2: /HS -> Net-(J2-Pad2)
- R19 pad 1: Net-(J2-Pad14) -> Net-(DD21-Pad21)
- R19 pad 2: /VS -> Net-(R17-Pad2)
- R2 pad 2: Net-(DD5-Pad10) -> /video_gen/SR1
- R20 pad 1: VCC -> Net-(DD21-Pad20)
- R20 pad 2: /WEN -> Net-(J2-Pad2)
- R21 pad 1: VCC -> GND
- R21 pad 2: /CSL -> Net-(R21-Pad2)
- R3 pad 1: PUP1 -> VCC
- R3 pad 2: VCC -> Net-(R3-Pad2)
- R4 pad 1: PUP2 -> VCC
- R4 pad 2: VCC -> Net-(R4-Pad2)
- R5 pad 1: PUP3 -> VCC
- R5 pad 2: VCC -> Net-(DD1-Pad1)
- R6 pad 1: Net-(R12-Pad2) -> VCC
- R6 pad 2: /R -> Net-(DD3-Pad10)
- R7 pad 1: /VR -> VCC
- R7 pad 2: /IR -> Net-(DD10-Pad7)
- R8 pad 1: Net-(R14-Pad2) -> VCC
- R8 pad 2: /G -> MVP
Routing:
- net VCC: track 747.2 -> 332.9 mm, vias 35 -> 17
- net GND: track 1128.6 -> 728.2 mm, vias 207 -> 60
- net /X1: track 124.7 -> 0.00 mm, vias 4 -> 0
- net /video_gen/SR1: track 0.00 -> 100.6 mm
- net /video_gen/SR0: track 0.00 -> 95.8 mm
- net /VM4: track 117.1 -> 21.6 mm, vias 1 -> 0
- net /CLK: track 89.8 -> 0.00 mm, vias 5 -> 0
- net /X0: track 89.0 -> 0.00 mm, vias 2 -> 0
- net /CPX: track 0.00 -> 82.5 mm, vias 0 -> 5
- net /PFA: track 76.2 -> 0.00 mm, vias 1 -> 0
- net /PFC: track 71.6 -> 0.00 mm, vias 1 -> 0
- net /D7: track 71.1 -> 0.00 mm, vias 4 -> 0
- net /D1: track 70.6 -> 0.00 mm, vias 4 -> 0
- net /D3: track 70.5 -> 0.00 mm, vias 4 -> 0
- net /PF8: track 69.4 -> 0.00 mm
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- added copper zone on In1.Cu, net GND
- added copper zone on In2.Cu, net VCC
Other:
- copper layers 2 -> 4
- net class Default removed
- board text added: "Orion-NG, zx-pk.ru andreil, 2020"
- board text removed: "ATF22V10"
- board text removed: "Orion-NG, zx-pk.ru andreil, 2018"
- board text removed: "АП6 245"
- board text removed: "ИЕ18 163"
- board text removed: "ИР10 166"
- board text removed: "ИР23 374"
- board text removed: "ИР33 573"
- board text removed: "ТМ9 174"
